Commit message: Changed sign to joint6 in urdf centauro

File: centauro/urdf/centauro_upperbody.urdf (robot description, URDF)
Before this commit: robot centauro, 19 links, 18 joints
Joints:
- joint j_arm1_6: axis 0 1 0 -> 0 -1 0
- joint j_arm2_6: axis 0 -1 0 -> 0 1 0

Commit message: Changed back to original values centauro_upperbody.urdf, the correct urdf is *_new

File: centauro/urdf/centauro_upperbody.urdf (robot description, URDF)
Before this commit: robot centauro, 19 links, 18 joints
Joints:
- joint j_arm1_6: axis 0 -1 0 -> 0 1 0
- joint j_arm2_6: axis 0 1 0 -> 0 -1 0
