Commit message: Apparently working urdf

File: centauro/urdf/centauro_bonn_review.urdf (robot description, URDF)
Before this commit: robot centauro, 21 links, 20 joints
Links:
- removed link ft_arm1_7
- added link l_arm_ft, mass 0.3
Joints:
- removed joint ft_j_arm1_7
- added joint l_arm_ft_joint: type fixed, parent arm1_7, child l_arm_ft, origin xyz=0 0 -0.0255 rpy=0 0 0, axis 1 0 0, limit lower=0.0 upper=0.0 effort=5 velocity=4.0
- joint ft_j_arm2_7: type revolute -> fixed
- joint j_arm2_8: type revolute -> fixed

Commit message: Set hand as fixed, added it as controlled joint inside SRDF

File: centauro/urdf/centauro_bonn_review.urdf (robot description, URDF)
Before this commit: robot centauro, 19 links, 18 joints
Joints:
- joint j_arm1_8: type revolute -> fixed
