Commit message: Fixed velocity limits of lower body

File: centauro/urdf/centauro_full_body.urdf (robot description, URDF)
Before this commit: robot centauro, 33 links, 32 joints
Joints:
- joint knee_pitch_1: limit lower=-3.14 upper=3.14 effort=35000 velocity=600.5 -> lower=-3.14 upper=3.14 effort=35000 velocity=6.5
- joint knee_pitch_2: limit lower=-3.14 upper=3.14 effort=35000 velocity=600.5 -> lower=-3.14 upper=3.14 effort=35000 velocity=6.5
- joint knee_pitch_3: limit lower=-3.14 upper=3.14 effort=35000 velocity=600.5 -> lower=-3.14 upper=3.14 effort=35000 velocity=6.5
- joint knee_pitch_4: limit lower=-3.14 upper=3.14 effort=35000 velocity=600.5 -> lower=-3.14 upper=3.14 effort=35000 velocity=6.5
