Commit message: config files updated for CENTAURO.

File: centauro/urdf/centauro_full_with_imu.urdf (robot description, URDF)
Before this commit: robot centauro, 36 links, 35 joints
Links:
- removed link arm2_8
- added link ft_arm2, mass 0.15; collision mesh filename=package://centauro/centauro_urdf/meshes/link9.stl scale=0.001 0.001 -0.001; visual mesh filename=package://centauro/centauro_urdf/meshes/link9.stl scale=0.001 0.001 -0.001
Joints:
- removed joint j_arm2_8
- added joint j_ft_arm2: type fixed, parent arm2_7, child ft_arm2, origin xyz=0.0 0.0 -0.0405 rpy=0.0 3.14159265359 -1.5707963268, axis 1 0 0, limit lower=0.0 upper=0 effort=0 velocity=0

File: centauro/urdf/centauro_upper_body_updated_inertia.urdf (robot description, URDF)
Before this commit: robot centauro, 19 links, 18 joints
Links:
- removed link arm2_8
- added link ft_arm2, mass 0.15; collision mesh filename=package://centauro/centauro_urdf/meshes/link9.stl scale=0.001 0.001 -0.001; visual mesh filename=package://centauro/centauro_urdf/meshes/link9.stl scale=0.001 0.001 -0.001
Joints:
- removed joint j_arm2_8
- added joint j_ft_arm2: type fixed, parent arm2_7, child ft_arm2, origin xyz=0.0 0.0 -0.0405 rpy=0.0 3.14159265359 -1.5707963268, axis 1 0 0, limit lower=0.0 upper=0 effort=0 velocity=0
