Commit message: Merge branch 'alaurenzi_configs' of github.com:ADVRHumanoids/ADVR_shared into alaurenzi_configs
# Conflicts:
#	bigman/configs/config_walkman.yaml
#	centauro/configs/config_centauro.yaml

File: centauro/urdf/centauro_full_fixed_wheels.urdf (robot description, URDF)
Before this commit: robot centauro, 48 links, 47 joints
Joints:
- joint j_wheel_1: type continuous -> fixed
- joint j_wheel_2: type continuous -> fixed
- joint j_wheel_3: type continuous -> fixed
- joint j_wheel_4: type continuous -> fixed

File: centauro/urdf/centauro_lower_body_fixed_wheels.urdf (robot description, URDF)
Before this commit: robot centauro, 48 links, 47 joints
Links:
- removed link arm1_1
- removed link arm1_2
- removed link arm1_3
- removed link arm1_4
- removed link arm1_5
- removed link arm1_6
- removed link arm1_7
- removed link arm1_8
- removed link arm2_1
- removed link arm2_2
- removed link arm2_3
- removed link arm2_4
- removed link arm2_5
- removed link arm2_6
- removed link arm2_7
- removed link arm2_8
- removed link torso_2
Joints:
- removed joint j_arm1_1
- removed joint j_arm1_2
- removed joint j_arm1_3
- removed joint j_arm1_4
- removed joint j_arm1_5
- removed joint j_arm1_6
- removed joint j_arm1_7
- removed joint j_arm1_8
- removed joint j_arm2_1
- removed joint j_arm2_2
- removed joint j_arm2_3
- removed joint j_arm2_4
- removed joint j_arm2_5
- removed joint j_arm2_6
- removed joint j_arm2_7
- removed joint j_arm2_8
- removed joint torso_yaw
- joint j_wheel_1: type continuous -> fixed
- joint j_wheel_2: type continuous -> fixed
- joint j_wheel_3: type continuous -> fixed
- joint j_wheel_4: type continuous -> fixed
