Commit message: config for floating base

File: centauro/urdf/centauro_upper_body_updated_inertia.urdf (robot description, URDF)
Before this commit: robot centauro, 19 links, 18 joints
Links:
- added link imu_link, mass 0.0
- added link left_arm_ft
- added link right_arm_ft
Joints:
- added joint imu_joint: type fixed, parent torso_2, child imu_link, origin xyz=-0.0704 0.0 -0.0416
- added joint l_arm_ft_joint: type fixed, parent arm1_7, child left_arm_ft, origin xyz=0 0 -0.0565 rpy=0 0 0
- added joint r_arm_ft_joint: type fixed, parent arm2_7, child right_arm_ft, origin xyz=0 0 -0.0565 rpy=0 0 0
