Commit message: change centauro to have only 14 joints

File: centauro/urdf/centauro_floating_arm.urdf (robot description, URDF)
Before this commit: robot centauro, 20 links, 19 joints
Links:
- added link left_arm_ft
- added link right_arm_ft
- link arm1_8: mass 0.1 -> 0.01
- link arm2_8: mass 0.1 -> 0.01
Joints:
- added joint l_arm_ft_joint: type fixed, parent arm1_7, child left_arm_ft, origin xyz=0 0 -0.0565 rpy=0 0 0
- added joint r_arm_ft_joint: type fixed, parent arm2_7, child right_arm_ft, origin xyz=0 0 -0.0565 rpy=0 0 0
- joint floating_base: origin (none) -> xyz=0.0 0.0 0.6 rpy=0 0 0; type floating -> fixed
- joint j_arm1_1: limit lower=-3.403 upper=1.658 effort=147 velocity=5.7 -> lower=-3.0 upper=3.0 effort=147 velocity=5.7
- joint j_arm1_2: limit lower=-3.49 upper=0 effort=147 velocity=5.7 -> lower=-3.0 upper=3.0 effort=147 velocity=5.7
- joint j_arm1_3: limit lower=-2.618 upper=2.618 effort=147 velocity=8.2 -> lower=-3.0 upper=3.0 effort=147 velocity=5.7
- joint j_arm1_4: limit lower=-2.530 upper=0.349 effort=147 velocity=8.2 -> lower=-3.0 upper=3.0 effort=147 velocity=5.7
- joint j_arm1_5: limit lower=-2.618 upper=2.618 effort=55 velocity=11.6 -> lower=-3.0 upper=3.0 effort=147 velocity=5.7
- joint j_arm1_6: limit lower=-1.570 upper=1.570 effort=55 velocity=11.6 -> lower=-3.0 upper=3.0 effort=147 velocity=5.7
- joint j_arm1_7: limit lower=-2.618 upper=2.618 effort=27 velocity=20.3 -> lower=-3.0 upper=3.0 effort=147 velocity=5.7
- joint j_arm1_8: origin xyz=0 0 -0.05 rpy=0 0 0.5 -> xyz=0 0 -0.05 rpy=0 0 0
- joint j_arm2_1: limit lower=-1.658 upper=3.403 effort=147 velocity=5.7 -> lower=-3.0 upper=3.0 effort=147 velocity=5.7
- joint j_arm2_2: limit lower=0 upper=3.49 effort=147 velocity=5.7 -> lower=-3.0 upper=3.0 effort=147 velocity=5.7
- joint j_arm2_3: limit lower=-2.618 upper=2.618 effort=147 velocity=8.2 -> lower=-3.0 upper=3.0 effort=147 velocity=5.7
- joint j_arm2_4: limit lower=-0.349 upper=2.530 effort=147 velocity=8.2 -> lower=-3.0 upper=3.0 effort=147 velocity=5.7
- joint j_arm2_5: limit lower=-2.618 upper=2.618 effort=55 velocity=11.6 -> lower=-3.0 upper=3.0 effort=147 velocity=5.7
- joint j_arm2_6: limit lower=-1.570 upper=1.570 effort=55 velocity=11.6 -> lower=-3.0 upper=3.0 effort=147 velocity=5.7
- joint j_arm2_7: limit lower=-2.618 upper=2.618 effort=27 velocity=20.3 -> lower=-3.0 upper=3.0 effort=147 velocity=5.7
- joint j_arm2_8: origin xyz=0 0 -0.05 rpy=0 0 -0.5 -> xyz=0 0 -0.05 rpy=0 0 0
