Commit message: Using latest Malgorzata URDF

File: centauro/urdf/centauro_lower_body_fixed_wheels_ARTURO.urdf (robot description, URDF)
Before this commit: robot centauro, 26 links, 25 joints
Links:
- added link foot_fl, mass 0; visual box size=0.01 0.01 0.01
- added link foot_fr, mass 0; visual box size=0.01 0.01 0.01
- added link foot_hl, mass 0; visual box size=0.01 0.01 0.01
- added link foot_hr, mass 0; visual box size=0.01 0.01 0.01
- added link imu_link, mass 0.0
Joints:
- added joint imu_joint: type fixed, parent pelvis, child imu_link, origin xyz=-0.0704 0.0 -0.0416
- added joint j_foot_fl: type fixed, parent ankle2_1, child foot_fl, origin xyz=0.0 0.0 0.30 rpy=0.0 0.0 0.0
- added joint j_foot_fr: type fixed, parent ankle2_2, child foot_fr, origin xyz=0.0 0.0 0.30 rpy=0.0 0.0 0.0
- added joint j_foot_hl: type fixed, parent ankle2_3, child foot_hl, origin xyz=0.0 0.0 0.30 rpy=0.0 0.0 0.0
- added joint j_foot_hr: type fixed, parent ankle2_4, child foot_hr, origin xyz=0.0 0.0 0.30 rpy=0.0 0.0 0.0
