Commit message: Added neck and velodyne.

File: centauro/urdf/centauro_no_head.urdf (robot description, URDF)
Before this commit: robot centauro, 47 links, 46 joints
Links:
- removed link neck_1
- removed link neck_2
- removed link neck_3
- added link foot_fl, mass 0; visual box size=0.01 0.01 0.01
- added link foot_fr, mass 0; visual box size=0.01 0.01 0.01
- added link foot_hl, mass 0; visual box size=0.01 0.01 0.01
- added link foot_hr, mass 0; visual box size=0.01 0.01 0.01
- link torso_2: mass 6.1886404 -> 4.5494226
Joints:
- removed joint neck_pitch
- removed joint neck_velodyne
- removed joint neck_yaw
- added joint j_foot_fl: type fixed, parent ankle2_1, child foot_fl, origin xyz=0.0 0.0 0.30 rpy=0.0 0.0 0.0
- added joint j_foot_fr: type fixed, parent ankle2_2, child foot_fr, origin xyz=0.0 0.0 0.30 rpy=0.0 0.0 0.0
- added joint j_foot_hl: type fixed, parent ankle2_3, child foot_hl, origin xyz=0.0 0.0 0.30 rpy=0.0 0.0 0.0
- added joint j_foot_hr: type fixed, parent ankle2_4, child foot_hr, origin xyz=0.0 0.0 0.30 rpy=0.0 0.0 0.0
- joint hip_yaw_1: limit lower=-1.13446401 upper=2.70526034 effort=304 velocity=8.8 -> lower=-0.78539816 upper=2.35619449 effort=304 velocity=8.8; origin xyz=0.25 0.125 -0.0566 rpy=3.14159265359 0.0 0.50709869865 -> xyz=0.225 0.125 0.11 rpy=3.14159265359 0.0 0.50709869865
- joint hip_yaw_2: limit lower=-2.70526034 upper=1.13446401 effort=304 velocity=8.8 -> lower=-2.35619449 upper=0.78539816 effort=304 velocity=8.8; origin xyz=0.25 -0.125 -0.0566 rpy=3.14159265359 0.0 -0.50709869865 -> xyz=0.225 -0.125 0.11 rpy=3.14159265359 0.0 -0.50709869865
- joint hip_yaw_3: limit lower=-2.70526034 upper=1.13446401 effort=304 velocity=8.8 -> lower=-2.35619449 upper=0.78539816 effort=304 velocity=8.8; origin xyz=-0.25 0.125 -0.0566 rpy=3.14159265359 0.0 2.63449395494 -> xyz=-0.225 0.125 0.11 rpy=3.14159265359 0.0 2.63449395494
- joint hip_yaw_4: limit lower=-1.13446401 upper=2.70526034 effort=304 velocity=8.8 -> lower=-0.78539816 upper=2.35619449 effort=304 velocity=8.8; origin xyz=-0.25 -0.125 -0.0566 rpy=3.14159265359 0.0 3.64869135224 -> xyz=-0.225 -0.125 0.11 rpy=3.14159265359 0.0 3.64869135224
- joint imu_joint: origin xyz=0.0 0.0 0.0 rpy=0.0 0.0 0.0 -> xyz=-0.0704 0.0 -0.0416
- joint j_arm1_1: origin xyz=0.04576 0.169137 0.116626 rpy=0.0 0.0 -0.523602668986 -> xyz=0.04576 0.169137 0.190626 rpy=0.0 0.0 -0.523602668986
- joint j_arm2_1: origin xyz=0.04576 -0.169137 0.116626 rpy=0.0 0.0 0.523602668986 -> xyz=0.04576 -0.169137 0.190626 rpy=0.0 0.0 0.523602668986
- joint reference: origin xyz=0.0 0.0 0.9256 -> xyz=0.0 0.0 0.759
- joint torso_yaw: origin xyz=0.2 0.0 0.256 -> xyz=0.175 0.0 0.36
