Commit message: Updated hip yaw ranges

File: centauro/urdf/centauro_full_wheels.urdf (robot description, URDF)
Before this commit: robot centauro, 52 links, 51 joints
Joints:
- joint hip_yaw_1: limit lower=-0.78539816 upper=2.35619449 effort=304 velocity=8.8 -> lower=-1.13446401 upper=2.70526034 effort=304 velocity=8.8
- joint hip_yaw_2: limit lower=-2.35619449 upper=0.78539816 effort=304 velocity=8.8 -> lower=-2.70526034 upper=1.13446401 effort=304 velocity=8.8
- joint hip_yaw_3: limit lower=-2.35619449 upper=0.78539816 effort=304 velocity=8.8 -> lower=-2.70526034 upper=1.13446401 effort=304 velocity=8.8
- joint hip_yaw_4: limit lower=-0.78539816 upper=2.35619449 effort=304 velocity=8.8 -> lower=-1.13446401 upper=2.70526034 effort=304 velocity=8.8
- joint imu_joint: origin xyz=-0.0704 0.0 -0.0416 -> xyz=0.0 0.0 0.0 rpy=0.0 0.0 0.0

Commit message: Better orientation of feet fixed joints

File: centauro/urdf/centauro_full_wheels.urdf (robot description, URDF)
Before this commit: robot centauro, 52 links, 51 joints
Joints:
- joint j_foot_fl: origin xyz=0.0 0.0 0.30 rpy=0.0 0.0 0.0 -> xyz=0.0 0.0 0.30 rpy=3.1415 0.0 3.1415
- joint j_foot_fr: origin xyz=0.0 0.0 0.30 rpy=0.0 0.0 0.0 -> xyz=0.0 0.0 0.30 rpy=3.1415 0.0 0.0
- joint j_foot_hl: origin xyz=0.0 0.0 0.30 rpy=0.0 0.0 0.0 -> xyz=0.0 0.0 0.30 rpy=3.1415 0.0 3.1415
- joint j_foot_hr: origin xyz=0.0 0.0 0.30 rpy=0.0 0.0 0.0 -> xyz=0.0 0.0 0.30 rpy=3.1415 0.0 0.0
