Commit message: FT added to the feet

File: centauro/urdf/centauro_lower_body_fixed_wheels.urdf (robot description, URDF)
Before this commit: robot centauro, 31 links, 30 joints
Links:
- added link fl_foot_ft, mass 0; visual box size=0.01 0.01 0.01
- added link fr_foot_ft, mass 0; visual box size=0.01 0.01 0.01
- added link hl_foot_ft, mass 0; visual box size=0.01 0.01 0.01
- added link hr_foot_ft, mass 0; visual box size=0.01 0.01 0.01
Joints:
- added joint j_fl_foot_ft: type fixed, parent ankle2_1, child fl_foot_ft, origin xyz=0 0 0 rpy=0 0 0
- added joint j_fr_foot_ft: type fixed, parent ankle2_2, child fr_foot_ft, origin xyz=0 0 0 rpy=0 0 0
- added joint j_hl_foot_ft: type fixed, parent ankle2_3, child hl_foot_ft, origin xyz=0 0 0 rpy=0 0 0
- added joint j_hr_foot_ft: type fixed, parent ankle2_4, child hr_foot_ft, origin xyz=0 0 0 rpy=0 0 0

Commit message: CONFIG/URDF/SRDF updated and tested on real hardware lower body + wheels

File: centauro/urdf/centauro_lower_body_fixed_wheels.urdf (robot description, URDF)
Before this commit: robot centauro, 26 links, 25 joints
Joints:
- joint j_wheel_1: limit effort=35 velocity=20.0 -> lower=-1000000000000000 upper=1000000000000000 effort=35 velocity=20.0; type fixed -> revolute
- joint j_wheel_2: limit effort=35 velocity=20.0 -> lower=-1000000000000000 upper=1000000000000000 effort=35 velocity=20.0; type fixed -> revolute
- joint j_wheel_3: limit effort=35 velocity=20.0 -> lower=-1000000000000000 upper=1000000000000000 effort=35 velocity=20.0; type fixed -> revolute
- joint j_wheel_4: limit effort=35 velocity=20.0 -> lower=-1000000000000000 upper=1000000000000000 effort=35 velocity=20.0; type fixed -> revolute

Commit message: Manual merge from devel to master.

File: centauro/urdf/centauro_lower_body_fixed_wheels.urdf (robot description, URDF)
Before this commit: robot centauro, 53 links, 52 joints
Links:
- removed link arm1_1
- removed link arm1_2
- removed link arm1_3
- removed link arm1_4
- removed link arm1_5
- removed link arm1_6
- removed link arm1_7
- removed link arm1_8
- removed link arm2_1
- removed link arm2_2
- removed link arm2_3
- removed link arm2_4
- removed link arm2_5
- removed link arm2_6
- removed link arm2_7
- removed link arm2_8
- removed link foot_fl
- removed link foot_fr
- removed link foot_hl
- removed link foot_hr
- removed link ft_arm1
- removed link ft_arm2
- removed link imu_link
- removed link neck_1
- removed link neck_2
- removed link neck_3
- removed link torso_2
Joints:
- removed joint imu_joint
- removed joint j_arm1_1
- removed joint j_arm1_2
- removed joint j_arm1_3
- removed joint j_arm1_4
- removed joint j_arm1_5
- removed joint j_arm1_6
- removed joint j_arm1_7
- removed joint j_arm1_8
- removed joint j_arm2_1
- removed joint j_arm2_2
- removed joint j_arm2_3
- removed joint j_arm2_4
- removed joint j_arm2_5
- removed joint j_arm2_6
- removed joint j_arm2_7
- removed joint j_arm2_8
- removed joint j_foot_fl
- removed joint j_foot_fr
- removed joint j_foot_hl
- removed joint j_foot_hr
- removed joint j_ft_arm1
- removed joint j_ft_arm2
- removed joint neck_pitch
- removed joint neck_velodyne
- removed joint neck_yaw
- removed joint torso_yaw
- joint hip_yaw_1: limit lower=-1.13446401 upper=2.70526034 effort=304 velocity=8.8 -> lower=-0.78539816 upper=2.35619449 effort=304 velocity=8.8; origin xyz=0.25 0.125 -0.0566 rpy=3.14159265359 0.0 0.50709869865 -> xyz=0.225 0.125 0.11 rpy=3.14159265359 0.0 0.50709869865
- joint hip_yaw_2: limit lower=-2.70526034 upper=1.13446401 effort=304 velocity=8.8 -> lower=-2.35619449 upper=0.78539816 effort=304 velocity=8.8; origin xyz=0.25 -0.125 -0.0566 rpy=3.14159265359 0.0 -0.50709869865 -> xyz=0.225 -0.125 0.11 rpy=3.14159265359 0.0 -0.50709869865
- joint hip_yaw_3: limit lower=-2.70526034 upper=1.13446401 effort=304 velocity=8.8 -> lower=-2.35619449 upper=0.78539816 effort=304 velocity=8.8; origin xyz=-0.25 0.125 -0.0566 rpy=3.14159265359 0.0 2.63449395494 -> xyz=-0.225 0.125 0.11 rpy=3.14159265359 0.0 2.63449395494
- joint hip_yaw_4: limit lower=-1.13446401 upper=2.70526034 effort=304 velocity=8.8 -> lower=-0.78539816 upper=2.35619449 effort=304 velocity=8.8; origin xyz=-0.25 -0.125 -0.0566 rpy=3.14159265359 0.0 3.64869135224 -> xyz=-0.225 -0.125 0.11 rpy=3.14159265359 0.0 3.64869135224
- joint j_wheel_1: type continuous -> revolute
- joint j_wheel_2: type continuous -> revolute
- joint j_wheel_3: type continuous -> revolute
- joint j_wheel_4: type continuous -> revolute
- joint reference: origin xyz=0.0 0.0 0.9256 -> xyz=0.0 0.0 0.759

File: centauro/urdf/centauro_no_head.urdf (robot description, URDF)
Before this commit: robot centauro, 53 links, 52 joints
Links:
- removed link ft_arm1
- removed link ft_arm2
- removed link neck_1
- removed link neck_2
- removed link neck_3
- link torso_2: mass 6.1886404 -> 4.5494226
Joints:
- removed joint j_ft_arm1
- removed joint j_ft_arm2
- removed joint neck_pitch
- removed joint neck_velodyne
- removed joint neck_yaw
- joint hip_yaw_1: limit lower=-1.13446401 upper=2.70526034 effort=304 velocity=8.8 -> lower=-0.78539816 upper=2.35619449 effort=304 velocity=8.8; origin xyz=0.25 0.125 -0.0566 rpy=3.14159265359 0.0 0.50709869865 -> xyz=0.225 0.125 0.11 rpy=3.14159265359 0.0 0.50709869865
- joint hip_yaw_2: limit lower=-2.70526034 upper=1.13446401 effort=304 velocity=8.8 -> lower=-2.35619449 upper=0.78539816 effort=304 velocity=8.8; origin xyz=0.25 -0.125 -0.0566 rpy=3.14159265359 0.0 -0.50709869865 -> xyz=0.225 -0.125 0.11 rpy=3.14159265359 0.0 -0.50709869865
- joint hip_yaw_3: limit lower=-2.70526034 upper=1.13446401 effort=304 velocity=8.8 -> lower=-2.35619449 upper=0.78539816 effort=304 velocity=8.8; origin xyz=-0.25 0.125 -0.0566 rpy=3.14159265359 0.0 2.63449395494 -> xyz=-0.225 0.125 0.11 rpy=3.14159265359 0.0 2.63449395494
- joint hip_yaw_4: limit lower=-1.13446401 upper=2.70526034 effort=304 velocity=8.8 -> lower=-0.78539816 upper=2.35619449 effort=304 velocity=8.8; origin xyz=-0.25 -0.125 -0.0566 rpy=3.14159265359 0.0 3.64869135224 -> xyz=-0.225 -0.125 0.11 rpy=3.14159265359 0.0 3.64869135224
- joint imu_joint: origin xyz=0.0 0.0 0.0 rpy=0.0 0.0 0.0 -> xyz=-0.0704 0.0 -0.0416
- joint j_arm1_1: origin xyz=0.04576 0.169137 0.116626 rpy=0.0 0.0 -0.523602668986 -> xyz=0.04576 0.169137 0.190626 rpy=0.0 0.0 -0.523602668986
- joint j_arm1_2: limit lower=-3.49 upper=-0.25 effort=147 velocity=5.7 -> lower=-3.49 upper=0 effort=147 velocity=5.7
- joint j_arm2_1: origin xyz=0.04576 -0.169137 0.116626 rpy=0.0 0.0 0.523602668986 -> xyz=0.04576 -0.169137 0.190626 rpy=0.0 0.0 0.523602668986
- joint j_arm2_2: limit lower=0.25 upper=3.49 effort=147 velocity=5.7 -> lower=0 upper=3.49 effort=147 velocity=5.7
- joint j_foot_fl: origin xyz=0.0 0.0 0.30 rpy=3.1415 0.0 3.1415 -> xyz=0.0 0.0 0.30 rpy=0.0 0.0 0.0
- joint j_foot_fr: origin xyz=0.0 0.0 0.30 rpy=3.1415 0.0 0.0 -> xyz=0.0 0.0 0.30 rpy=0.0 0.0 0.0
- joint j_foot_hl: origin xyz=0.0 0.0 0.30 rpy=3.1415 0.0 3.1415 -> xyz=0.0 0.0 0.30 rpy=0.0 0.0 0.0
- joint j_foot_hr: origin xyz=0.0 0.0 0.30 rpy=3.1415 0.0 0.0 -> xyz=0.0 0.0 0.30 rpy=0.0 0.0 0.0
- joint j_wheel_1: type continuous -> revolute
- joint j_wheel_2: type continuous -> revolute
- joint j_wheel_3: type continuous -> revolute
- joint j_wheel_4: type continuous -> revolute
- joint reference: origin xyz=0.0 0.0 0.9256 -> xyz=0.0 0.0 0.759
- joint torso_yaw: origin xyz=0.2 0.0 0.256 -> xyz=0.175 0.0 0.36

File: cogimon/urdf/cogimon_imu.urdf (robot description, URDF)
Before this commit: robot cogimon, 36 links, 35 joints
Links:
- added link imu_link, mass 0
Joints:
- added joint imu_joint: type fixed, parent Waist, child imu_link, origin xyz=0 0 0 rpy=0 0 0
