Commit message: working simulation fixing the issue of the wheels.

File: centauro/urdf/centauro.urdf (robot description, URDF)
Before this commit: robot centauro, 48 links, 47 joints
Joints:
- joint j_wheel_1: limit lower=-1000000000000000 upper=1000000000000000 effort=35 velocity=20.0 -> (none); type revolute -> fixed
- joint j_wheel_2: limit lower=-1000000000000000 upper=1000000000000000 effort=35 velocity=20.0 -> (none); type revolute -> fixed
- joint j_wheel_3: limit lower=-1000000000000000 upper=1000000000000000 effort=35 velocity=20.0 -> (none); type revolute -> fixed
- joint j_wheel_4: limit lower=-1000000000000000 upper=1000000000000000 effort=35 velocity=20.0 -> (none); type revolute -> fixed

Commit message: working version with left hand and left FT.

File: centauro/urdf/centauro.urdf (robot description, URDF)
Before this commit: robot centauro, 47 links, 46 joints
Links:
- added link ft_arm1, mass 0.15; collision mesh filename=package://centauro/centauro_urdf/meshes/link9.stl scale=0.001 0.001 -0.001; visual mesh filename=package://centauro/centauro_urdf/meshes/link9.stl scale=0.001 0.001 -0.001
- added link ft_arm2, mass 0.15; collision mesh filename=package://centauro/centauro_urdf/meshes/link9.stl scale=0.001 0.001 -0.001; visual mesh filename=package://centauro/centauro_urdf/meshes/link9.stl scale=0.001 0.001 -0.001
Joints:
- added joint j_ft_arm1: type fixed, parent arm1_7, child ft_arm1, origin xyz=0.0 0.0 -0.0405 rpy=0.0 3.14159265359 -1.5707963268, axis 1 0 0, limit lower=0.0 upper=0 effort=0 velocity=0
- added joint j_ft_arm2: type fixed, parent arm2_7, child ft_arm2, origin xyz=0.0 0.0 -0.0405 rpy=0.0 3.14159265359 -1.5707963268, axis 1 0 0, limit lower=0.0 upper=0 effort=0 velocity=0

Commit message: continuos

File: centauro/urdf/centauro.urdf (robot description, URDF)
Before this commit: robot centauro, 49 links, 48 joints
Joints:
- joint j_wheel_1: type revolute -> continuous
- joint j_wheel_2: type revolute -> continuous
- joint j_wheel_3: type revolute -> continuous
- joint j_wheel_4: type revolute -> continuous

Commit message: vel continuous

File: centauro/urdf/centauro.urdf (robot description, URDF)
Before this commit: robot centauro, 49 links, 48 joints
Joints:
- joint neck_velodyne: type revolute -> continuous

Commit message: Working version of ALEX integration: manually setting higher limits on j_arm*_2

File: centauro/urdf/centauro.urdf (robot description, URDF)
Before this commit: robot centauro, 49 links, 48 joints
Joints:
- joint j_arm1_2: limit lower=-3.49 upper=0 effort=147 velocity=5.7 -> lower=-3.49 upper=-0.25 effort=147 velocity=5.7
- joint j_arm2_2: limit lower=0 upper=3.49 effort=147 velocity=5.7 -> lower=0.25 upper=3.49 effort=147 velocity=5.7

Commit message: set wheels + velodyne as continuous joint urdf

File: centauro/urdf/centauro.urdf (robot description, URDF)
Before this commit: robot centauro, 49 links, 48 joints
Joints:
- joint j_wheel_1: type revolute -> continuous
- joint j_wheel_2: type revolute -> continuous
- joint j_wheel_3: type revolute -> continuous
- joint j_wheel_4: type revolute -> continuous
- joint neck_velodyne: type revolute -> continuous

Commit message: Feet fixed links

File: centauro/urdf/centauro.urdf (robot description, URDF)
Before this commit: robot centauro, 49 links, 48 joints
Links:
- added link foot_fl, mass 0; visual box size=0.01 0.01 0.01
- added link foot_fr, mass 0; visual box size=0.01 0.01 0.01
- added link foot_hl, mass 0; visual box size=0.01 0.01 0.01
- added link foot_hr, mass 0; visual box size=0.01 0.01 0.01
Joints:
- added joint j_foot_fl: type fixed, parent ankle2_1, child foot_fl, origin xyz=0.0 0.0 0.30 rpy=3.1415 0.0 3.1415
- added joint j_foot_fr: type fixed, parent ankle2_2, child foot_fr, origin xyz=0.0 0.0 0.30 rpy=3.1415 0.0 0.0
- added joint j_foot_hl: type fixed, parent ankle2_3, child foot_hl, origin xyz=0.0 0.0 0.30 rpy=3.1415 0.0 3.1415
- added joint j_foot_hr: type fixed, parent ankle2_4, child foot_hr, origin xyz=0.0 0.0 0.30 rpy=3.1415 0.0 0.0

Commit message: FIxed FT

File: centauro/urdf/centauro.urdf (robot description, URDF)
Before this commit: robot centauro, 49 links, 48 joints
Joints:
- joint j_ft_arm1: origin xyz=0.0 0.0 -0.0405 rpy=0.0 3.14159265359 -1.5707963268 -> xyz=0.0 0.0 -0.0405 rpy=0.0 3.14159265359 -3.14159265359
- joint j_ft_arm2: origin xyz=0.0 0.0 -0.0405 rpy=0.0 3.14159265359 -1.5707963268 -> xyz=0.0 0.0 -0.0405 rpy=0.0 3.14159265359 -3.14159265359

Commit message: Updating urdf for centauro

File: centauro/urdf/centauro.urdf (robot description, URDF)
Before this commit: robot centauro, 47 links, 46 joints
Links:
- added link foot_fl, mass 0; visual box size=0.01 0.01 0.01
- added link foot_fr, mass 0; visual box size=0.01 0.01 0.01
- added link foot_hl, mass 0; visual box size=0.01 0.01 0.01
- added link foot_hr, mass 0; visual box size=0.01 0.01 0.01
- added link ft_arm1, mass 0.15; collision mesh filename=package://centauro/centauro_urdf/meshes/link9.stl scale=0.001 0.001 -0.001; visual mesh filename=package://centauro/centauro_urdf/meshes/link9.stl scale=0.001 0.001 -0.001
- added link ft_arm2, mass 0.15; collision mesh filename=package://centauro/centauro_urdf/meshes/link9.stl scale=0.001 0.001 -0.001; visual mesh filename=package://centauro/centauro_urdf/meshes/link9.stl scale=0.001 0.001 -0.001
Joints:
- added joint j_foot_fl: type fixed, parent ankle2_1, child foot_fl, origin xyz=0.0 0.0 0.30 rpy=3.1415 0.0 3.1415
- added joint j_foot_fr: type fixed, parent ankle2_2, child foot_fr, origin xyz=0.0 0.0 0.30 rpy=3.1415 0.0 0.0
- added joint j_foot_hl: type fixed, parent ankle2_3, child foot_hl, origin xyz=0.0 0.0 0.30 rpy=3.1415 0.0 3.1415
- added joint j_foot_hr: type fixed, parent ankle2_4, child foot_hr, origin xyz=0.0 0.0 0.30 rpy=3.1415 0.0 0.0
- added joint j_ft_arm1: type fixed, parent arm1_7, child ft_arm1, origin xyz=0.0 0.0 -0.0405 rpy=0.0 3.14159265359 -1.5707963268, axis 1 0 0, limit lower=0.0 upper=0 effort=0 velocity=0
- added joint j_ft_arm2: type fixed, parent arm2_7, child ft_arm2, origin xyz=0.0 0.0 -0.0405 rpy=0.0 3.14159265359 -1.5707963268, axis 1 0 0, limit lower=0.0 upper=0 effort=0 velocity=0
- joint j_arm1_2: limit lower=-3.49 upper=0 effort=147 velocity=5.7 -> lower=-3.49 upper=-0.25 effort=147 velocity=5.7
- joint j_arm2_2: limit lower=0 upper=3.49 effort=147 velocity=5.7 -> lower=0.25 upper=3.49 effort=147 velocity=5.7
- joint j_wheel_1: type revolute -> continuous
- joint j_wheel_2: type revolute -> continuous
- joint j_wheel_3: type revolute -> continuous
- joint j_wheel_4: type revolute -> continuous
- joint neck_velodyne: type revolute -> continuous

Commit message: Centauro configs coherent with xbotcore_ft_compatible branch of centauro-simulator

File: centauro/urdf/centauro.urdf (robot description, URDF)
Before this commit: robot centauro, 53 links, 52 joints
Links:
- removed link foot_fl
- removed link foot_fr
- removed link foot_hl
- removed link foot_hr
- added link camera_central, mass 0.1
- added link camera_left, mass 0.1
- added link camera_right, mass 0.1
- added link ft_foot_1, mass 0
- added link ft_foot_2, mass 0
- added link ft_foot_3, mass 0
- added link ft_foot_4, mass 0
- added link kinect, mass 0.1
- added link kinect2_rgb_optical_frame
- added link velodyne_mount, mass 0.1
- link ft_arm1: geometry 
- link ft_arm2: geometry 
Joints:
- removed joint j_foot_fl
- removed joint j_foot_fr
- removed joint j_foot_hl
- removed joint j_foot_hr
- removed joint j_ft_arm1
- removed joint j_ft_arm2
- added joint j_camera_central: type fixed, parent torso_2, child camera_central, origin xyz=0.0559593 5e-12 0.390626 rpy=0.0 0.349065586018 0.0
- added joint j_camera_left: type fixed, parent torso_2, child camera_left, origin xyz=0.0191392 0.0525845 0.390626 rpy=0.0 0.349065586018 1.2217302006
- added joint j_camera_right: type fixed, parent torso_2, child camera_right, origin xyz=0.0191392 -0.0525845 0.390626 rpy=0.0 0.349065586018 -1.2217302006
- added joint j_ft_1: type fixed, parent arm1_7, child ft_arm1, origin xyz=0.0 0.0 -0.0405 rpy=0.0 3.14159265359 -3.14159265359, axis 0 0 1, limit lower=0.0 upper=0.0 effort=0 velocity=0
- added joint j_ft_2: type fixed, parent arm2_7, child ft_arm2, origin xyz=0.0 0.0 -0.0405 rpy=0.0 3.14159265359 -3.14159265359, axis 0 0 1, limit lower=0.0 upper=0.0 effort=0 velocity=0
- added joint j_ft_foot_1: type fixed, parent ankle2_1, child ft_foot_1, origin xyz=0.0 0.00085 0.23735 rpy=0 0 0
- added joint j_ft_foot_2: type fixed, parent ankle2_2, child ft_foot_2, origin xyz=0.0 0.00085 0.23735 rpy=0 0 0
- added joint j_ft_foot_3: type fixed, parent ankle2_3, child ft_foot_3, origin xyz=0.0 0.00085 0.23735 rpy=0 0 0
- added joint j_ft_foot_4: type fixed, parent ankle2_4, child ft_foot_4, origin xyz=0.0 0.00085 0.23735 rpy=0 0 0
- added joint j_kinect: type fixed, parent neck_2, child kinect, origin xyz=0.03 -0.0596 0.045855 rpy=0.0 0.0 0.0
- added joint j_kinect_optical_frame: type fixed, parent kinect, child kinect2_rgb_optical_frame, origin xyz=0.050 -0.110 -0.035 rpy= -1.5707963268 0 -1.5707963268
- added joint j_velodyne: type fixed, parent neck_3, child velodyne_mount, origin xyz=-0.138 0.0 -0.033 rpy=0.0 0.0 -3.14159265359
- joint hip_pitch_1: origin xyz=0.0 0.0 0.059 rpy=1.57079632679 0.0 0.50709869865 -> xyz=0.0 0.0 0.0625 rpy=1.57079632679 0.0 0.46141612323
- joint hip_pitch_2: origin xyz=0.0 0.0 0.059 rpy=1.57079632679 0.0 2.63449395494 -> xyz=0.0 0.0 0.0625 rpy=1.57079632679 0.0 2.68017653036
- joint hip_pitch_3: origin xyz=0.0 0.0 0.059 rpy=1.57079632679 0.0 2.63449395494 -> xyz=0.0 0.0 0.0625 rpy=1.57079632679 0.0 2.68017653036
- joint hip_pitch_4: origin xyz=0.0 0.0 0.059 rpy=1.57079632679 0.0 0.50709869865 -> xyz=0.0 0.0 0.0625 rpy=1.57079632679 0.0 0.46141612323
- joint hip_yaw_1: origin xyz=0.25 0.125 -0.0566 rpy=3.14159265359 0.0 0.50709869865 -> xyz=0.25 0.125 -0.0566 rpy=3.14159265359 0.0 0.461416123228
- joint hip_yaw_2: origin xyz=0.25 -0.125 -0.0566 rpy=3.14159265359 0.0 -0.50709869865 -> xyz=0.25 -0.125 -0.0566 rpy=3.14159265359 0.0 -0.461416123228
- joint hip_yaw_3: origin xyz=-0.25 0.125 -0.0566 rpy=3.14159265359 0.0 2.63449395494 -> xyz=-0.25 0.125 -0.0566 rpy=3.14159265359 0.0 2.68017653036
- joint hip_yaw_4: origin xyz=-0.25 -0.125 -0.0566 rpy=3.14159265359 0.0 3.64869135224 -> xyz=-0.25 -0.125 -0.0566 rpy=3.14159265359 0.0 3.60300877682
- joint j_arm1_2: limit lower=-3.49 upper=-0.25 effort=147 velocity=5.7 -> lower=-3.49 upper=0 effort=147 velocity=5.7
- joint j_arm1_8: limit lower=0.0 upper=0 effort=0 velocity=0 -> (none); origin xyz=0.0 0.0 -0.0405 rpy=0.0 3.14159265359 -1.5707963268 -> xyz=0.0 0.0 0.0 rpy=0.0 0.0 -1.5707963268; parent arm1_7 -> ft_arm1
- joint j_arm2_2: limit lower=0.25 upper=3.49 effort=147 velocity=5.7 -> lower=0 upper=3.49 effort=147 velocity=5.7
- joint j_arm2_8: limit lower=0.0 upper=0 effort=0 velocity=0 -> (none); origin xyz=0.0 0.0 -0.0405 rpy=0.0 3.14159265359 -1.5707963268 -> xyz=0.0 0.0 0.0 rpy=0.0 0.0 -1.5707963268; parent arm2_7 -> ft_arm2
- joint j_wheel_1: limit lower=-1000000000000000 upper=1000000000000000 effort=35 velocity=20.0 -> effort=35 velocity=20.0; origin xyz=0.0 0.00085 0.235 rpy=1.57079632679 0.0 0.0 -> xyz=0.0 0.00085 0.23735 rpy=1.57079632679 0.0 3.14159265359
- joint j_wheel_2: limit lower=-1000000000000000 upper=1000000000000000 effort=35 velocity=20.0 -> effort=35 velocity=20.0; origin xyz=0.0 0.00085 0.235 rpy=1.57079632679 0.0 0.0 -> xyz=0.0 0.00085 0.23735 rpy=1.57079632679 0.0 3.14159265359
- joint j_wheel_3: limit lower=-1000000000000000 upper=1000000000000000 effort=35 velocity=20.0 -> effort=35 velocity=20.0; origin xyz=0.0 0.00085 0.235 rpy=1.57079632679 0.0 0.0 -> xyz=0.0 0.00085 0.23735 rpy=1.57079632679 0.0 3.14159265359
- joint j_wheel_4: limit lower=-1000000000000000 upper=1000000000000000 effort=35 velocity=20.0 -> effort=35 velocity=20.0; origin xyz=0.0 0.00085 0.235 rpy=1.57079632679 0.0 0.0 -> xyz=0.0 0.00085 0.23735 rpy=1.57079632679 0.0 3.14159265359
- joint neck_velodyne: limit lower=-1000000000000000 upper=1000000000000000 effort=35 velocity=5.7 -> effort=35 velocity=5.7
- joint reference: origin xyz=0.0 0.0 0.9256 -> xyz=0.0 0.0 0.93445
