Commit message: simplified mesh centauro urdf

File: centauro/urdf/centauro.urdf (robot description, URDF)
Before this commit: robot centauro, 53 links, 52 joints
Links:
- link ankle1_1: geometry collision mesh filename=package://centauro/centauro_urdf/meshes/convex_hull/ankle-p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 scale=0.001 0.001 0.001; visual mesh filename=package://centauro/centauro_urdf/meshes/simplified/ankle-pi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 scale=0.001 0.001 0.001
- link ankle1_2: geometry collision mesh filename=package://centauro/centauro_urdf/meshes/convex_hull/ankle-p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 scale=0.001 0.001 0.001; visual mesh filename=package://centauro/centauro_urdf/meshes/simplified/ankle-pi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 scale=0.001 0.001 0.001
- link ankle1_3: geometry collision mesh filename=package://centauro/centauro_urdf/meshes/convex_hull/ankle-p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 scale=0.001 0.001 0.001; visual mesh filename=package://centauro/centauro_urdf/meshes/simplified/ankle-pi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 scale=0.001 0.001 0.001
- link ankle1_4: geometry collision mesh filename=package://centauro/centauro_urdf/meshes/convex_hull/ankle-p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 scale=0.001 0.001 0.001; visual mesh filename=package://centauro/centauro_urdf/meshes/simplified/ankle-pi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 scale=0.001 0.001 0.001
- link ankle2_1: geometry collision mesh filename=package://centauro/centauro_urdf/meshes/convex_hull/ankle-y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 scale=0.001 0.001 0.001; visual mesh filename=package://centauro/centauro_urdf/meshes/simplified/ankle-ya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 scale=0.001 0.001 0.001
- link ankle2_2: geometry collision mesh filename=package://centauro/centauro_urdf/meshes/convex_hull/ankle-y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 scale=0.001 0.001 0.001; visual mesh filename=package://centauro/centauro_urdf/meshes/simplified/ankle-ya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 scale=0.001 0.001 0.001
- link ankle2_3: geometry collision mesh filename=package://centauro/centauro_urdf/meshes/convex_hull/ankle-y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 scale=0.001 0.001 0.001; visual mesh filename=package://centauro/centauro_urdf/meshes/simplified/ankle-ya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 scale=0.001 0.001 0.001
- link ankle2_4: geometry collision mesh filename=package://centauro/centauro_urdf/meshes/convex_hull/ankle-y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 scale=0.001 0.001 0.001; visual mesh filename=package://centauro/centauro_urdf/meshes/simplified/ankle-ya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 scale=0.001 0.001 0.001
- link arm1_1: geometry collision mesh filename=package://centauro/centauro_urdf/meshes/convex_hull/link2.s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 scale=0.001 -0.001 0.001; visual mesh filename=package://centauro/centauro_urdf/meshes/simplified/link2.stl scale=0.001 -0.001 0.001
- link arm1_2: geometry collision mesh filename=package://centauro/centauro_urdf/meshes/convex_hull/link3.s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 scale=0.001 -0.001 0.001; visual mesh filename=package://centauro/centauro_urdf/meshes/simplified/link3.stl scale=0.001 -0.001 0.001
- link arm1_3: geometry collision mesh filename=package://centauro/centauro_urdf/meshes/convex_hull/link4.s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 scale=0.001 -0.001 0.001; visual mesh filename=package://centauro/centauro_urdf/meshes/simplified/link4.stl scale=0.001 -0.001 0.001
- link arm1_4: geometry collision mesh filename=package://centauro/centauro_urdf/meshes/convex_hull/link5.s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 scale=0.001 -0.001 0.001; visual mesh filename=package://centauro/centauro_urdf/meshes/simplified/link5.stl scale=0.001 -0.001 0.001
- link arm1_5: geometry collision mesh filename=package://centauro/centauro_urdf/meshes/convex_hull/link6.s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 scale=0.001 -0.001 0.001; visual mesh filename=package://centauro/centauro_urdf/meshes/simplified/link6.stl scale=0.001 -0.001 0.001
- link arm1_6: geometry collision mesh filename=package://centauro/centauro_urdf/meshes/convex_hull/link7.s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 scale=0.001 -0.001 0.001; visual mesh filename=package://centauro/centauro_urdf/meshes/simplified/link7.stl scale=0.001 -0.001 0.001
- link arm1_7: geometry collision mesh filename=package://centauro/centauro_urdf/meshes/convex_hull/link8.s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 scale=0.001 -0.001 0.001; visual mesh filename=package://centauro/centauro_urdf/meshes/simplified/link8.stl scale=0.001 -0.001 0.001
- link arm1_8: geometry collision mesh filename=package://centauro/centauro_urdf/meshes/convex_hull/link9.s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 scale=0.001 -0.001 -0.001; visual mesh filename=package://centauro/centauro_urdf/meshes/simplified/link9.stl scale=0.001 -0.001 -0.001
- link arm2_1: geometry collision mesh filename=package://centauro/centauro_urdf/meshes/convex_hull/link2.s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 scale=0.001 0.001 0.001; visual mesh filename=package://centauro/centauro_urdf/meshes/simplified/link2.stl scale=0.001 0.001 0.001
- link arm2_2: geometry collision mesh filename=package://centauro/centauro_urdf/meshes/convex_hull/link3.s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 scale=0.001 0.001 0.001; visual mesh filename=package://centauro/centauro_urdf/meshes/simplified/link3.stl scale=0.001 0.001 0.001
- link arm2_3: geometry collision mesh filename=package://centauro/centauro_urdf/meshes/convex_hull/link4.s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 scale=0.001 0.001 0.001; visual mesh filename=package://centauro/centauro_urdf/meshes/simplified/link4.stl scale=0.001 0.001 0.001
- link arm2_4: geometry collision mesh filename=package://centauro/centauro_urdf/meshes/convex_hull/link5.s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 scale=0.001 0.001 0.001; visual mesh filename=package://centauro/centauro_urdf/meshes/simplified/link5.stl scale=0.001 0.001 0.001
- link arm2_5: geometry collision mesh filename=package://centauro/centauro_urdf/meshes/convex_hull/link6.s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 scale=0.001 0.001 0.001; visual mesh filename=package://centauro/centauro_urdf/meshes/simplified/link6.stl scale=0.001 0.001 0.001
- link arm2_6: geometry collision mesh filename=package://centauro/centauro_urdf/meshes/convex_hull/link7.s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 scale=0.001 0.001 0.001; visual mesh filename=package://centauro/centauro_urdf/meshes/simplified/link7.stl scale=0.001 0.001 0.001
- link arm2_7: geometry collision mesh filename=package://centauro/centauro_urdf/meshes/convex_hull/link8.s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 scale=0.001 0.001 0.001; visual mesh filename=package://centauro/centauro_urdf/meshes/simplified/link8.stl scale=0.001 0.001 0.001
- link arm2_8: geometry collision mesh filename=package://centauro/centauro_urdf/meshes/convex_hull/link9.s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 scale=0.001 0.001 -0.001; visual mesh filename=package://centauro/centauro_urdf/meshes/simplified/link9.stl scale=0.001 0.001 -0.001
- link ft_arm1: geometry collision mesh filename=package://centauro/centauro_urdf/meshes/link9.stl scale=0.001 0.001 -0.001; visual mesh filename=package://centauro/centauro_urdf/meshes/simplified/link9.stl scale=0.001 0.001 -0.001
- link ft_arm2: geometry collision mesh filename=package://centauro/centauro_urdf/meshes/link9.stl scale=0.001 0.001 -0.001; visual mesh filename=package://centauro/centauro_urdf/meshes/simplified/link9.stl scale=0.001 0.001 -0.001
- link hip1_1: geometry collision mesh filename=package://centauro/centauro_urdf/meshes/convex_hull/hip-yaw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 scale=0.001 0.001 0.001; visual mesh filename=package://centauro/centauro_urdf/meshes/simplified/hip-yaw.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 scale=0.001 0.001 0.001
- link hip1_2: geometry collision mesh filename=package://centauro/centauro_urdf/meshes/convex_hull/hip-yaw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 scale=0.001 0.001 0.001; visual mesh filename=package://centauro/centauro_urdf/meshes/simplified/hip-yaw.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 scale=0.001 0.001 0.001
- link hip1_3: geometry collision mesh filename=package://centauro/centauro_urdf/meshes/convex_hull/hip-yaw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 scale=0.001 0.001 0.001; visual mesh filename=package://centauro/centauro_urdf/meshes/simplified/hip-yaw.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 scale=0.001 0.001 0.001
- link hip1_4: geometry collision mesh filename=package://centauro/centauro_urdf/meshes/convex_hull/hip-yaw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 scale=0.001 0.001 0.001; visual mesh filename=package://centauro/centauro_urdf/meshes/simplified/hip-yaw.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 scale=0.001 0.001 0.001
- link hip2_1: geometry collision mesh filename=package://centauro/centauro_urdf/meshes/convex_hull/hip-pit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 scale=0.001 0.001 0.001; visual mesh filename=package://centauro/centauro_urdf/meshes/simplified/hip-pitc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 scale=0.001 0.001 0.001
- link hip2_2: geometry collision mesh filename=package://centauro/centauro_urdf/meshes/convex_hull/hip-pit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 scale=0.001 0.001 0.001; visual mesh filename=package://centauro/centauro_urdf/meshes/simplified/hip-pitc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 scale=0.001 0.001 0.001
- link hip2_3: geometry collision mesh filename=package://centauro/centauro_urdf/meshes/convex_hull/hip-pit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 scale=0.001 0.001 0.001; visual mesh filename=package://centauro/centauro_urdf/meshes/simplified/hip-pitc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 scale=0.001 0.001 0.001
- link hip2_4: geometry collision mesh filename=package://centauro/centauro_urdf/meshes/convex_hull/hip-pit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 scale=0.001 0.001 0.001; visual mesh filename=package://centauro/centauro_urdf/meshes/simplified/hip-pitc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 scale=0.001 0.001 0.001
- link knee_1: geometry collision mesh filename=package://centauro/centauro_urdf/meshes/convex_hull/knee.stl scale=0.001 0.001 0.001; visual mesh filename=package://centauro/centauro_urdf/meshes/simplified/knee.stl scale=0.001 0.001 0.001
- link knee_2: geometry collision mesh filename=package://centauro/centauro_urdf/meshes/convex_hull/knee.stl scale=0.001 0.001 0.001; visual mesh filename=package://centauro/centauro_urdf/meshes/simplified/knee.stl scale=0.001 0.001 0.001
- link knee_3: geometry collision mesh filename=package://centauro/centauro_urdf/meshes/convex_hull/knee.stl scale=0.001 0.001 0.001; visual mesh filename=package://centauro/centauro_urdf/meshes/simplified/knee.stl scale=0.001 0.001 0.001
- link knee_4: geometry collision mesh filename=package://centauro/centauro_urdf/meshes/convex_hull/knee.stl scale=0.001 0.001 0.001; visual mesh filename=package://centauro/centauro_urdf/meshes/simplified/knee.stl scale=0.001 0.001 0.001
- link neck_1: geometry collision mesh filename=package://centauro/centauro_urdf/meshes/convex_hull/neck_ya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 scale=0.001 0.001 0.001; visual mesh filename=package://centauro/centauro_urdf/meshes/simplified/neck_yaw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 scale=0.001 0.001 0.001
- link neck_2: geometry collision mesh filename=package://centauro/centauro_urdf/meshes/convex_hull/neck_pi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 scale=0.001 0.001 0.001; visual mesh filename=package://centauro/centauro_urdf/meshes/simplified/neck_pit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 scale=0.001 0.001 0.001
- link neck_3: geometry collision mesh filename=package://centauro/centauro_urdf/meshes/convex_hull/velodyn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 scale=0.001 0.001 0.001; visual mesh filename=package://centauro/centauro_urdf/meshes/simplified/velodyne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 scale=0.001 0.001 0.001
- link pelvis: geometry collision mesh filename=package://centauro/centauro_urdf/meshes/convex_hull/pelvis.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 scale=0.001 0.001 0.001; visual mesh filename=package://centauro/centauro_urdf/meshes/simplified/pelvis.s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 scale=0.001 0.001 0.001
- link torso_2: geometry collision mesh filename=package://centauro/centauro_urdf/meshes/convex_hull/link1.s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 scale=0.001 0.001 0.001; visual mesh filename=package://centauro/centauro_urdf/meshes/simplified/link1.stl scale=0.001 0.001 0.001
- link wheel_1: geometry collision mesh filename=package://centauro/centauro_urdf/meshes/convex_hull/wheel.s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 scale=0.001 0.001 0.001; visual mesh filename=package://centauro/centauro_urdf/meshes/simplified/wheel.stl scale=0.001 0.001 0.001
- link wheel_2: geometry collision mesh filename=package://centauro/centauro_urdf/meshes/convex_hull/wheel.s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 scale=0.001 0.001 0.001; visual mesh filename=package://centauro/centauro_urdf/meshes/simplified/wheel.stl scale=0.001 0.001 0.001
- link wheel_3: geometry collision mesh filename=package://centauro/centauro_urdf/meshes/convex_hull/wheel.s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 scale=0.001 0.001 0.001; visual mesh filename=package://centauro/centauro_urdf/meshes/simplified/wheel.stl scale=0.001 0.001 0.001
- link wheel_4: geometry collision mesh filename=package://centauro/centauro_urdf/meshes/convex_hull/wheel.s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 scale=0.001 0.001 0.001; visual mesh filename=package://centauro/centauro_urdf/meshes/simplified/wheel.stl scale=0.001 0.001 0.001
