Commit message: latest set of experiment with HERI hand and new low level working

File: centauro/urdf/centauro.urdf (robot description, URDF)
Before this commit: robot centauro, 53 links, 52 joints
Links:
- added link HeriDown_link, mass 2.0
- added link HeriEnd_link, mass 2.0
- added link HeriUp_link, mass 2.0
- link ankle1_1: geometry collision mesh filename=package://centauro/centauro_urdf/meshes/convex_hull/ankle-p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 scale=0.001 0.001 0.001; visual mesh filename=package://centauro/centauro_urdf/meshes/simplified/ankle-pi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 scale=0.001 0.001 0.001
- link ankle1_2: geometry collision mesh filename=package://centauro/centauro_urdf/meshes/convex_hull/ankle-p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 scale=0.001 0.001 0.001; visual mesh filename=package://centauro/centauro_urdf/meshes/simplified/ankle-pi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 scale=0.001 0.001 0.001
- link ankle1_3: geometry collision mesh filename=package://centauro/centauro_urdf/meshes/convex_hull/ankle-p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 scale=0.001 0.001 0.001; visual mesh filename=package://centauro/centauro_urdf/meshes/simplified/ankle-pi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 scale=0.001 0.001 0.001
- link ankle1_4: geometry collision mesh filename=package://centauro/centauro_urdf/meshes/convex_hull/ankle-p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 scale=0.001 0.001 0.001; visual mesh filename=package://centauro/centauro_urdf/meshes/simplified/ankle-pi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 scale=0.001 0.001 0.001
- link ankle2_1: geometry collision mesh filename=package://centauro/centauro_urdf/meshes/convex_hull/ankle-y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 scale=0.001 0.001 0.001; visual mesh filename=package://centauro/centauro_urdf/meshes/simplified/ankle-ya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 scale=0.001 0.001 0.001
- link ankle2_2: geometry collision mesh filename=package://centauro/centauro_urdf/meshes/convex_hull/ankle-y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 scale=0.001 0.001 0.001; visual mesh filename=package://centauro/centauro_urdf/meshes/simplified/ankle-ya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 scale=0.001 0.001 0.001
- link ankle2_3: geometry collision mesh filename=package://centauro/centauro_urdf/meshes/convex_hull/ankle-y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 scale=0.001 0.001 0.001; visual mesh filename=package://centauro/centauro_urdf/meshes/simplified/ankle-ya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 scale=0.001 0.001 0.001
- link ankle2_4: geometry collision mesh filename=package://centauro/centauro_urdf/meshes/convex_hull/ankle-y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 scale=0.001 0.001 0.001; visual mesh filename=package://centauro/centauro_urdf/meshes/simplified/ankle-ya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 scale=0.001 0.001 0.001
- link arm1_1: geometry collision mesh filename=package://centauro/centauro_urdf/meshes/convex_hull/link2.s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 scale=0.001 -0.001 0.001; visual mesh filename=package://centauro/centauro_urdf/meshes/simplified/link2.stl scale=0.001 -0.001 0.001
- link arm1_2: geometry collision mesh filename=package://centauro/centauro_urdf/meshes/convex_hull/link3.s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 scale=0.001 -0.001 0.001; visual mesh filename=package://centauro/centauro_urdf/meshes/simplified/link3.stl scale=0.001 -0.001 0.001
- link arm1_3: geometry collision mesh filename=package://centauro/centauro_urdf/meshes/convex_hull/link4.s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 scale=0.001 -0.001 0.001; visual mesh filename=package://centauro/centauro_urdf/meshes/simplified/link4.stl scale=0.001 -0.001 0.001
- link arm1_4: geometry collision mesh filename=package://centauro/centauro_urdf/meshes/convex_hull/link5.s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 scale=0.001 -0.001 0.001; visual mesh filename=package://centauro/centauro_urdf/meshes/simplified/link5.stl scale=0.001 -0.001 0.001
- link arm1_5: geometry collision mesh filename=package://centauro/centauro_urdf/meshes/convex_hull/link6.s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 scale=0.001 -0.001 0.001; visual mesh filename=package://centauro/centauro_urdf/meshes/simplified/link6.stl scale=0.001 -0.001 0.001
- link arm1_6: geometry collision mesh filename=package://centauro/centauro_urdf/meshes/convex_hull/link7.s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 scale=0.001 -0.001 0.001; visual mesh filename=package://centauro/centauro_urdf/meshes/simplified/link7.stl scale=0.001 -0.001 0.001
- link arm1_7: geometry collision mesh filename=package://centauro/centauro_urdf/meshes/convex_hull/link8.s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 scale=0.001 -0.001 0.001; visual mesh filename=package://centauro/centauro_urdf/meshes/simplified/link8.stl scale=0.001 -0.001 0.001
- link arm1_8: geometry collision mesh filename=package://centauro/centauro_urdf/meshes/convex_hull/link9.s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 scale=0.001 -0.001 -0.001; visual mesh filename=package://centauro/centauro_urdf/meshes/simplified/link9.stl scale=0.001 -0.001 -0.001
- link arm2_1: geometry collision mesh filename=package://centauro/centauro_urdf/meshes/convex_hull/link2.s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 scale=0.001 0.001 0.001; visual mesh filename=package://centauro/centauro_urdf/meshes/simplified/link2.stl scale=0.001 0.001 0.001
- link arm2_2: geometry collision mesh filename=package://centauro/centauro_urdf/meshes/convex_hull/link3.s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 scale=0.001 0.001 0.001; visual mesh filename=package://centauro/centauro_urdf/meshes/simplified/link3.stl scale=0.001 0.001 0.001
- link arm2_3: geometry collision mesh filename=package://centauro/centauro_urdf/meshes/convex_hull/link4.s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 scale=0.001 0.001 0.001; visual mesh filename=package://centauro/centauro_urdf/meshes/simplified/link4.stl scale=0.001 0.001 0.001
- link arm2_4: geometry collision mesh filename=package://centauro/centauro_urdf/meshes/convex_hull/link5.s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 scale=0.001 0.001 0.001; visual mesh filename=package://centauro/centauro_urdf/meshes/simplified/link5.stl scale=0.001 0.001 0.001
- link arm2_5: geometry collision mesh filename=package://centauro/centauro_urdf/meshes/convex_hull/link6.s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 scale=0.001 0.001 0.001; visual mesh filename=package://centauro/centauro_urdf/meshes/simplified/link6.stl scale=0.001 0.001 0.001
- link arm2_6: geometry collision mesh filename=package://centauro/centauro_urdf/meshes/convex_hull/link7.s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 scale=0.001 0.001 0.001; visual mesh filename=package://centauro/centauro_urdf/meshes/simplified/link7.stl scale=0.001 0.001 0.001
- link arm2_7: geometry collision mesh filename=package://centauro/centauro_urdf/meshes/convex_hull/link8.s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 scale=0.001 0.001 0.001; visual mesh filename=package://centauro/centauro_urdf/meshes/simplified/link8.stl scale=0.001 0.001 0.001
- link arm2_8: geometry collision mesh filename=package://centauro/centauro_urdf/meshes/convex_hull/link9.s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 scale=0.001 0.001 -0.001; visual mesh filename=package://centauro/centauro_urdf/meshes/simplified/link9.stl scale=0.001 0.001 -0.001
- link ft_arm1: geometry collision mesh filename=package://centauro/centauro_urdf/meshes/link9.stl scale=0.001 0.001 -0.001; visual mesh filename=package://centauro/centauro_urdf/meshes/simplified/link9.stl scale=0.001 0.001 -0.001
- link ft_arm2: geometry collision mesh filename=package://centauro/centauro_urdf/meshes/link9.stl scale=0.001 0.001 -0.001; visual mesh filename=package://centauro/centauro_urdf/meshes/simplified/link9.stl scale=0.001 0.001 -0.001
- link hip1_1: geometry collision mesh filename=package://centauro/centauro_urdf/meshes/convex_hull/hip-yaw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 scale=0.001 0.001 0.001; visual mesh filename=package://centauro/centauro_urdf/meshes/simplified/hip-yaw.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 scale=0.001 0.001 0.001
- link hip1_2: geometry collision mesh filename=package://centauro/centauro_urdf/meshes/convex_hull/hip-yaw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 scale=0.001 0.001 0.001; visual mesh filename=package://centauro/centauro_urdf/meshes/simplified/hip-yaw.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 scale=0.001 0.001 0.001
- link hip1_3: geometry collision mesh filename=package://centauro/centauro_urdf/meshes/convex_hull/hip-yaw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 scale=0.001 0.001 0.001; visual mesh filename=package://centauro/centauro_urdf/meshes/simplified/hip-yaw.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 scale=0.001 0.001 0.001
- link hip1_4: geometry collision mesh filename=package://centauro/centauro_urdf/meshes/convex_hull/hip-yaw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 scale=0.001 0.001 0.001; visual mesh filename=package://centauro/centauro_urdf/meshes/simplified/hip-yaw.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 scale=0.001 0.001 0.001
- link hip2_1: geometry collision mesh filename=package://centauro/centauro_urdf/meshes/convex_hull/hip-pit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 scale=0.001 0.001 0.001; visual mesh filename=package://centauro/centauro_urdf/meshes/simplified/hip-pitc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 scale=0.001 0.001 0.001
- link hip2_2: geometry collision mesh filename=package://centauro/centauro_urdf/meshes/convex_hull/hip-pit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 scale=0.001 0.001 0.001; visual mesh filename=package://centauro/centauro_urdf/meshes/simplified/hip-pitc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 scale=0.001 0.001 0.001
- link hip2_3: geometry collision mesh filename=package://centauro/centauro_urdf/meshes/convex_hull/hip-pit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 scale=0.001 0.001 0.001; visual mesh filename=package://centauro/centauro_urdf/meshes/simplified/hip-pitc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 scale=0.001 0.001 0.001
- link hip2_4: geometry collision mesh filename=package://centauro/centauro_urdf/meshes/convex_hull/hip-pit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 scale=0.001 0.001 0.001; visual mesh filename=package://centauro/centauro_urdf/meshes/simplified/hip-pitc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 scale=0.001 0.001 0.001
- link knee_1: geometry collision mesh filename=package://centauro/centauro_urdf/meshes/convex_hull/knee.stl scale=0.001 0.001 0.001; visual mesh filename=package://centauro/centauro_urdf/meshes/simplified/knee.stl scale=0.001 0.001 0.001
- link knee_2: geometry collision mesh filename=package://centauro/centauro_urdf/meshes/convex_hull/knee.stl scale=0.001 0.001 0.001; visual mesh filename=package://centauro/centauro_urdf/meshes/simplified/knee.stl scale=0.001 0.001 0.001
- link knee_3: geometry collision mesh filename=package://centauro/centauro_urdf/meshes/convex_hull/knee.stl scale=0.001 0.001 0.001; visual mesh filename=package://centauro/centauro_urdf/meshes/simplified/knee.stl scale=0.001 0.001 0.001
- link knee_4: geometry collision mesh filename=package://centauro/centauro_urdf/meshes/convex_hull/knee.stl scale=0.001 0.001 0.001; visual mesh filename=package://centauro/centauro_urdf/meshes/simplified/knee.stl scale=0.001 0.001 0.001
- link neck_1: geometry collision mesh filename=package://centauro/centauro_urdf/meshes/convex_hull/neck_ya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 scale=0.001 0.001 0.001; visual mesh filename=package://centauro/centauro_urdf/meshes/simplified/neck_yaw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 scale=0.001 0.001 0.001
- link neck_2: geometry collision mesh filename=package://centauro/centauro_urdf/meshes/convex_hull/neck_pi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 scale=0.001 0.001 0.001; visual mesh filename=package://centauro/centauro_urdf/meshes/simplified/neck_pit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 scale=0.001 0.001 0.001
- link neck_3: geometry collision mesh filename=package://centauro/centauro_urdf/meshes/convex_hull/velodyn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 scale=0.001 0.001 0.001; visual mesh filename=package://centauro/centauro_urdf/meshes/simplified/velodyne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 scale=0.001 0.001 0.001
- link pelvis: geometry collision mesh filename=package://centauro/centauro_urdf/meshes/convex_hull/pelvis.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 scale=0.001 0.001 0.001; visual mesh filename=package://centauro/centauro_urdf/meshes/simplified/pelvis.s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 scale=0.001 0.001 0.001
- link torso_2: geometry collision mesh filename=package://centauro/centauro_urdf/meshes/convex_hull/link1.s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 scale=0.001 0.001 0.001; visual mesh filename=package://centauro/centauro_urdf/meshes/simplified/link1.stl scale=0.001 0.001 0.001
- link wheel_1: geometry collision mesh filename=package://centauro/centauro_urdf/meshes/convex_hull/wheel.s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 scale=0.001 0.001 0.001; visual mesh filename=package://centauro/centauro_urdf/meshes/simplified/wheel.stl scale=0.001 0.001 0.001
- link wheel_2: geometry collision mesh filename=package://centauro/centauro_urdf/meshes/convex_hull/wheel.s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 scale=0.001 0.001 0.001; visual mesh filename=package://centauro/centauro_urdf/meshes/simplified/wheel.stl scale=0.001 0.001 0.001
- link wheel_3: geometry collision mesh filename=package://centauro/centauro_urdf/meshes/convex_hull/wheel.s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 scale=0.001 0.001 0.001; visual mesh filename=package://centauro/centauro_urdf/meshes/simplified/wheel.stl scale=0.001 0.001 0.001
- link wheel_4: geometry collision mesh filename=package://centauro/centauro_urdf/meshes/convex_hull/wheel.s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 scale=0.001 0.001 0.001; visual mesh filename=package://centauro/centauro_urdf/meshes/simplified/wheel.stl scale=0.001 0.001 0.001
Joints:
- added joint 110: type fixed, parent HeriDown_link, child HeriUp_link, origin xyz=0 0 0.11 rpy=0 0 0, axis 0 0 1
- added joint 111: type fixed, parent HeriUp_link, child HeriEnd_link, origin xyz=0 0 0.2005 rpy=0 0 0, axis 0 -1 0
- added joint HeriBase: type fixed, parent arm1_8, child HeriDown_link, origin xyz=0 0 0 rpy=0 0 0

Commit message: right z axis sign for CENTAURO wheels

File: centauro/urdf/centauro.urdf (robot description, URDF)
Before this commit: robot centauro, 53 links, 52 joints
Joints:
- joint j_wheel_1: axis 0 0 1 -> 0 0 -1
- joint j_wheel_2: axis 0 0 1 -> 0 0 -1
- joint j_wheel_3: axis 0 0 1 -> 0 0 -1
- joint j_wheel_4: axis 0 0 1 -> 0 0 -1

Commit message: XBot compliance

File: centauro/urdf/centauro.urdf (robot description, URDF)
Before this commit: robot centauro, 53 links, 52 joints
Links:
- removed link foot_fl
- removed link foot_fr
- removed link foot_hl
- removed link foot_hr
- added link camera_central, mass 0.1
- added link camera_left, mass 0.1
- added link camera_right, mass 0.1
- added link kinect, mass 0.1
- added link kinect2_rgb_optical_frame
- added link velodyne_mount, mass 0.1
- link arm1_8: mass 0.15 -> 1.8366865; geometry collision mesh filename=package://centauro/centauro_urdf/meshes/convex_hull/heri.stl scale=0.001 -0.001 -0.001; visual mesh filename=package://centauro/centauro_urdf/meshes/simplified/heri.stl scale=0.001 -0.001 -0.001
- link ft_arm1: geometry 
- link ft_arm2: geometry 
Joints:
- removed joint j_foot_fl
- removed joint j_foot_fr
- removed joint j_foot_hl
- removed joint j_foot_hr
- removed joint j_ft_arm1
- removed joint j_ft_arm2
- added joint j_camera_central: type fixed, parent torso_2, child camera_central, origin xyz=0.0559593 5e-12 0.390626 rpy=0.0 0.349065586018 0.0
- added joint j_camera_left: type fixed, parent torso_2, child camera_left, origin xyz=0.0191392 0.0525845 0.390626 rpy=0.0 0.349065586018 1.2217302006
- added joint j_camera_right: type fixed, parent torso_2, child camera_right, origin xyz=0.0191392 -0.0525845 0.390626 rpy=0.0 0.349065586018 -1.2217302006
- added joint j_ft_1: type fixed, parent arm1_7, child ft_arm1, origin xyz=0.0 0.0 -0.0405 rpy=0.0 3.14159265359 -3.14159265359, axis 0 0 1, limit lower=0.0 upper=0.0 effort=0 velocity=0
- added joint j_ft_2: type fixed, parent arm2_7, child ft_arm2, origin xyz=0.0 0.0 -0.0405 rpy=0.0 3.14159265359 -3.14159265359, axis 0 0 1, limit lower=0.0 upper=0.0 effort=0 velocity=0
- added joint j_kinect: type fixed, parent neck_2, child kinect, origin xyz=0.03 -0.0596 0.045855 rpy=0.0 0.0 0.0
- added joint j_kinect_optical_frame: type fixed, parent kinect, child kinect2_rgb_optical_frame, origin xyz=0.050 -0.110 -0.035 rpy= -1.5707963268 0 -1.5707963268
- added joint j_velodyne: type fixed, parent neck_3, child velodyne_mount, origin xyz=-0.138 0.0 -0.033 rpy=0.0 0.0 -3.14159265359
- joint ankle_pitch_1: limit lower=-2.61799388 upper=2.61799388 effort=147 velocity=8.1 -> lower=-2.4056 upper=2.3184 effort=147 velocity=8.1
- joint ankle_pitch_2: limit lower=-2.61799388 upper=2.61799388 effort=147 velocity=8.1 -> lower=-2.3266 upper=2.3914 effort=147 velocity=8.1
- joint ankle_pitch_3: limit lower=-2.61799388 upper=2.61799388 effort=147 velocity=8.1 -> lower=-2.4696 upper=2.4464 effort=147 velocity=8.1
- joint ankle_pitch_4: limit lower=-2.61799388 upper=2.61799388 effort=147 velocity=8.1 -> lower=-2.3426 upper=2.3934 effort=147 velocity=8.1
- joint ankle_yaw_1: limit lower=-2.79252680 upper=2.79252680 effort=35 velocity=20.0 -> lower=-2.5626 upper=2.5384 effort=35 velocity=20.0
- joint ankle_yaw_2: limit lower=-2.79252680 upper=2.79252680 effort=35 velocity=20.0 -> lower=-2.5546 upper=2.5484 effort=35 velocity=20.0
- joint ankle_yaw_3: limit lower=-2.79252680 upper=2.79252680 effort=35 velocity=20.0 -> lower=-2.5606 upper=2.5454 effort=35 velocity=20.0
- joint ankle_yaw_4: limit lower=-2.79252680 upper=2.79252680 effort=35 velocity=20.0 -> lower=-2.6046 upper=2.5514 effort=35 velocity=20.0
- joint hip_pitch_1: limit lower=-2.09439510 upper=2.09439510 effort=304 velocity=8.8 -> lower=-2.0226 upper=2.02748 effort=304 velocity=8.8; origin xyz=0.0 0.0 0.059 rpy=1.57079632679 0.0 0.50709869865 -> xyz=0.0 0.0 0.0625 rpy=1.57079632679 0.0 0.46141612323
- joint hip_pitch_2: limit lower=-2.09439510 upper=2.09439510 effort=304 velocity=8.8 -> lower=-2.0156 upper=2.0354 effort=304 velocity=8.8; origin xyz=0.0 0.0 0.059 rpy=1.57079632679 0.0 2.63449395494 -> xyz=0.0 0.0 0.0625 rpy=1.57079632679 0.0 2.68017653036
- joint hip_pitch_3: limit lower=-2.09439510 upper=2.09439510 effort=304 velocity=8.8 -> lower=-2.0126 upper=2.0384 effort=304 velocity=8.8; origin xyz=0.0 0.0 0.059 rpy=1.57079632679 0.0 2.63449395494 -> xyz=0.0 0.0 0.0625 rpy=1.57079632679 0.0 2.68017653036
- joint hip_pitch_4: limit lower=-2.09439510 upper=2.09439510 effort=304 velocity=8.8 -> lower=-2.0326 upper=2.0524 effort=304 velocity=8.8; origin xyz=0.0 0.0 0.059 rpy=1.57079632679 0.0 0.50709869865 -> xyz=0.0 0.0 0.0625 rpy=1.57079632679 0.0 0.46141612323
- joint hip_yaw_1: limit lower=-1.13446401 upper=2.70526034 effort=304 velocity=8.8 -> lower=-0.9432 upper=2.5138 effort=304 velocity=8.8; origin xyz=0.25 0.125 -0.0566 rpy=3.14159265359 0.0 0.50709869865 -> xyz=0.25 0.125 -0.0566 rpy=3.14159265359 0.0 0.461416123228
- joint hip_yaw_2: limit lower=-2.70526034 upper=1.13446401 effort=304 velocity=8.8 -> lower=-2.511 upper=0.943 effort=304 velocity=8.8; origin xyz=0.25 -0.125 -0.0566 rpy=3.14159265359 0.0 -0.50709869865 -> xyz=0.25 -0.125 -0.0566 rpy=3.14159265359 0.0 -0.461416123228
- joint hip_yaw_3: limit lower=-2.70526034 upper=1.13446401 effort=304 velocity=8.8 -> lower=-2.51 upper=0.943 effort=304 velocity=8.8; origin xyz=-0.25 0.125 -0.0566 rpy=3.14159265359 0.0 2.63449395494 -> xyz=-0.25 0.125 -0.0566 rpy=3.14159265359 0.0 2.68017653036
- joint hip_yaw_4: limit lower=-1.13446401 upper=2.70526034 effort=304 velocity=8.8 -> lower=-0.9412 upper=2.5138 effort=304 velocity=8.8; origin xyz=-0.25 -0.125 -0.0566 rpy=3.14159265359 0.0 3.64869135224 -> xyz=-0.25 -0.125 -0.0566 rpy=3.14159265359 0.0 3.60300877682
- joint j_arm1_1: limit lower=-3.403 upper=1.658 effort=147 velocity=5.7 -> lower=-3.348 upper=1.578 effort=147 velocity=5.7
- joint j_arm1_2: limit lower=-3.49 upper=-0.25 effort=147 velocity=5.7 -> lower=-3.42 upper=-0.056 effort=147 velocity=5.7
- joint j_arm1_3: limit lower=-2.618 upper=2.618 effort=147 velocity=8.2 -> lower=-2.5556 upper=2.5424 effort=147 velocity=8.2
- joint j_arm1_4: limit lower=-2.530 upper=0.349 effort=147 velocity=8.2 -> lower=-2.4636 upper=0.2804 effort=147 velocity=8.2
- joint j_arm1_5: limit lower=-2.618 upper=2.618 effort=55 velocity=11.6 -> lower=-2.5406 upper=2.5534 effort=55 velocity=11.6
- joint j_arm1_6: limit lower=-1.570 upper=1.570 effort=55 velocity=11.6 -> lower=-1.5096 upper=1.5044 effort=55 velocity=11.6
- joint j_arm1_7: limit lower=-2.618 upper=2.618 effort=27 velocity=20.3 -> lower=-2.5376 upper=2.5554 effort=27 velocity=20.3
- joint j_arm1_8: limit lower=0.0 upper=0 effort=0 velocity=0 -> (none); origin xyz=0.0 0.0 -0.0405 rpy=0.0 3.14159265359 -1.5707963268 -> xyz=0.0 0.0 0.0 rpy=0.0 0.0 0.0; parent arm1_7 -> ft_arm1
- joint j_arm2_1: limit lower=-1.658 upper=3.403 effort=147 velocity=5.7 -> lower=-1.6102 upper=3.3138 effort=147 velocity=5.7
- joint j_arm2_2: limit lower=0.25 upper=3.49 effort=147 velocity=5.7 -> lower=0.0578 upper=3.4288 effort=147 velocity=5.7
- joint j_arm2_3: limit lower=-2.618 upper=2.618 effort=147 velocity=8.2 -> lower=-2.5426 upper=2.5524 effort=147 velocity=8.2
- joint j_arm2_4: limit lower=-0.349 upper=2.530 effort=147 velocity=8.2 -> lower=-0.2796 upper=2.4564 effort=147 velocity=8.2
- joint j_arm2_5: limit lower=-2.618 upper=2.618 effort=55 velocity=11.6 -> lower=-2.5626 upper=2.5464 effort=55 velocity=11.6
- joint j_arm2_6: limit lower=-1.570 upper=1.570 effort=55 velocity=11.6 -> lower=-1.4726 upper=1.5364 effort=55 velocity=11.6
- joint j_arm2_7: limit lower=-2.618 upper=2.618 effort=27 velocity=20.3 -> lower=-3.0908 upper=2.0114 effort=27 velocity=20.3
- joint j_arm2_8: limit lower=0.0 upper=0 effort=0 velocity=0 -> (none); origin xyz=0.0 0.0 -0.0405 rpy=0.0 3.14159265359 -1.5707963268 -> xyz=0.0 0.0 0.0 rpy=0.0 0.0 -1.5707963268; parent arm2_7 -> ft_arm2
- joint j_wheel_1: limit lower=-1000000000000000 upper=1000000000000000 effort=35 velocity=20.0 -> effort=35 velocity=20.0; origin xyz=0.0 0.00085 0.235 rpy=1.57079632679 0.0 0.0 -> xyz=0.0 0.00085 0.23735 rpy=1.57079632679 0.0 3.14159265359
- joint j_wheel_2: limit lower=-1000000000000000 upper=1000000000000000 effort=35 velocity=20.0 -> effort=35 velocity=20.0; origin xyz=0.0 0.00085 0.235 rpy=1.57079632679 0.0 0.0 -> xyz=0.0 0.00085 0.23735 rpy=1.57079632679 0.0 3.14159265359
- joint j_wheel_3: limit lower=-1000000000000000 upper=1000000000000000 effort=35 velocity=20.0 -> effort=35 velocity=20.0; origin xyz=0.0 0.00085 0.235 rpy=1.57079632679 0.0 0.0 -> xyz=0.0 0.00085 0.23735 rpy=1.57079632679 0.0 3.14159265359
- joint j_wheel_4: limit lower=-1000000000000000 upper=1000000000000000 effort=35 velocity=20.0 -> effort=35 velocity=20.0; origin xyz=0.0 0.00085 0.235 rpy=1.57079632679 0.0 0.0 -> xyz=0.0 0.00085 0.23735 rpy=1.57079632679 0.0 3.14159265359
- joint knee_pitch_1: limit lower=-2.61799388 upper=2.61799388 effort=304 velocity=8.8 -> lower=-2.4056 upper=2.3994 effort=304 velocity=8.8
- joint knee_pitch_2: limit lower=-2.61799388 upper=2.61799388 effort=304 velocity=8.8 -> lower=-2.4006 upper=2.4034 effort=304 velocity=8.8
- joint knee_pitch_3: limit lower=-2.61799388 upper=2.61799388 effort=304 velocity=8.8 -> lower=-2.4056 upper=2.4064 effort=304 velocity=8.8
- joint knee_pitch_4: limit lower=-2.61799388 upper=2.61799388 effort=304 velocity=8.8 -> lower=-2.4176 upper=2.3884 effort=304 velocity=8.8
- joint neck_velodyne: limit lower=-1000000000000000 upper=1000000000000000 effort=35 velocity=5.7 -> effort=35 velocity=5.7
- joint reference: origin xyz=0.0 0.0 0.9256 -> xyz=0.0 0.0 0.93445

Commit message: change the collision shape of knee kinks to cylinder as capsule of self-collision avoidance

File: centauro/urdf/centauro.urdf (robot description, URDF)
Before this commit: robot centauro, 53 links, 52 joints
Links:
- link hip2_3: geometry collision cylinder length=0.4 radius=0.05; visual mesh filename=package://centauro/centauro_urdf/meshes/hip-pitch.stl scale=0.001 0.001 0.001
- link hip2_4: geometry collision cylinder length=0.4 radius=0.05; visual mesh filename=package://centauro/centauro_urdf/meshes/hip-pitch.stl scale=0.001 0.001 0.001
- link knee_3: geometry collision cylinder length=0.25 radius=0.05; visual mesh filename=package://centauro/centauro_urdf/meshes/knee.stl scale=0.001 0.001 0.001
- link knee_4: geometry collision cylinder length=0.25 radius=0.05; visual mesh filename=package://centauro/centauro_urdf/meshes/knee.stl scale=0.001 0.001 0.001

Commit message: friday before change

File: centauro/urdf/centauro.urdf (robot description, URDF)
Before this commit: robot centauro, 55 links, 54 joints
Joints:
- joint reference: type floating -> fixed
