Commit message: Final Monday

File: centauro/urdf/centauro.urdf (robot description, URDF)
Before this commit: robot centauro, 55 links, 54 joints
Links:
- removed link ft_arm1
- removed link ft_arm2
- link ankle1_1: geometry collision box size=0.09 0.09 0.09; visual mesh filename=package://centauro/centauro_urdf/meshes/simplified/ankle-pi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 scale=0.001 0.001 0.001
- link ankle1_2: geometry collision box size=0.09 0.09 0.09; visual mesh filename=package://centauro/centauro_urdf/meshes/simplified/ankle-pi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 scale=0.001 0.001 0.001
- link ankle1_3: geometry collision box size=0.09 0.09 0.09; visual mesh filename=package://centauro/centauro_urdf/meshes/simplified/ankle-pi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 scale=0.001 0.001 0.001
- link ankle1_4: geometry collision box size=0.09 0.09 0.09; visual mesh filename=package://centauro/centauro_urdf/meshes/simplified/ankle-pi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 scale=0.001 0.001 0.001
- link ankle2_1: geometry collision box size=0.09 0.09 0.09; visual mesh filename=package://centauro/centauro_urdf/meshes/simplified/ankle-ya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 scale=0.001 0.001 0.001
- link ankle2_2: geometry collision box size=0.09 0.09 0.09; visual mesh filename=package://centauro/centauro_urdf/meshes/simplified/ankle-ya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 scale=0.001 0.001 0.001
- link ankle2_3: geometry collision box size=0.09 0.09 0.09; visual mesh filename=package://centauro/centauro_urdf/meshes/simplified/ankle-ya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 scale=0.001 0.001 0.001
- link ankle2_4: geometry collision box size=0.09 0.09 0.09; visual mesh filename=package://centauro/centauro_urdf/meshes/simplified/ankle-ya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 scale=0.001 0.001 0.001
- link arm1_1: geometry collision box size=0.05 0.1 0.05; visual mesh filename=package://centauro/centauro_urdf/meshes/simplified/link2.stl scale=0.001 -0.001 0.001
- link arm1_2: geometry collision box size=0.05 0.05 0.2; visual mesh filename=package://centauro/centauro_urdf/meshes/simplified/link3.stl scale=0.001 -0.001 0.001
- link arm1_3: geometry collision box size=0.05 0.05 0.10; visual mesh filename=package://centauro/centauro_urdf/meshes/simplified/link4.stl scale=0.001 -0.001 0.001
- link arm1_4: geometry collision box size=0.05 0.05 0.10; visual mesh filename=package://centauro/centauro_urdf/meshes/simplified/link5.stl scale=0.001 -0.001 0.001
- link arm1_5: geometry collision box size=0.05 0.05 0.1; visual mesh filename=package://centauro/centauro_urdf/meshes/simplified/link6.stl scale=0.001 -0.001 0.001
- link arm1_6: geometry collision box size=0.05 0.05 0.13; visual mesh filename=package://centauro/centauro_urdf/meshes/simplified/link7.stl scale=0.001 -0.001 0.001
- link arm1_7: geometry collision box size=0.05 0.05 0.05; visual mesh filename=package://centauro/centauro_urdf/meshes/simplified/link8.stl scale=0.001 -0.001 0.001
- link arm1_8: mass 1.8366865 -> 0.15; geometry collision cylinder length=0.13 radius=0.013; visual mesh filename=package://centauro/centauro_urdf/meshes/simplified/link9.stl scale=0.001 -0.001 -0.001
- link arm2_1: geometry collision box size=0.05 0.1 0.05; visual mesh filename=package://centauro/centauro_urdf/meshes/simplified/link2.stl scale=0.001 0.001 0.001
- link arm2_2: geometry collision box size=0.05 0.05 0.2; visual mesh filename=package://centauro/centauro_urdf/meshes/simplified/link3.stl scale=0.001 0.001 0.001
- link arm2_3: geometry collision box size=0.05 0.05 0.10; visual mesh filename=package://centauro/centauro_urdf/meshes/simplified/link4.stl scale=0.001 0.001 0.001
- link arm2_4: geometry collision box size=0.05 0.05 0.10; visual mesh filename=package://centauro/centauro_urdf/meshes/simplified/link5.stl scale=0.001 0.001 0.001
- link arm2_5: geometry collision box size=0.05 0.05 0.1; visual mesh filename=package://centauro/centauro_urdf/meshes/simplified/link6.stl scale=0.001 0.001 0.001
- link arm2_6: geometry collision box size=0.05 0.05 0.13; visual mesh filename=package://centauro/centauro_urdf/meshes/simplified/link7.stl scale=0.001 0.001 0.001
- link arm2_7: geometry collision box size=0.05 0.05 0.05; visual mesh filename=package://centauro/centauro_urdf/meshes/simplified/link8.stl scale=0.001 0.001 0.001
- link arm2_8: geometry collision cylinder length=0.13 radius=0.013; visual mesh filename=package://centauro/centauro_urdf/meshes/simplified/link9.stl scale=0.001 0.001 -0.001
- link hip1_1: geometry collision box size=0.05 0.05 0.05; visual mesh filename=package://centauro/centauro_urdf/meshes/simplified/hip-yaw.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 scale=0.001 0.001 0.001
- link hip1_2: geometry collision box size=0.05 0.05 0.05; visual mesh filename=package://centauro/centauro_urdf/meshes/simplified/hip-yaw.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 scale=0.001 0.001 0.001
- link hip1_3: geometry collision box size=0.05 0.05 0.05; visual mesh filename=package://centauro/centauro_urdf/meshes/simplified/hip-yaw.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 scale=0.001 0.001 0.001
- link hip1_4: geometry collision box size=0.05 0.05 0.05; visual mesh filename=package://centauro/centauro_urdf/meshes/simplified/hip-yaw.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 scale=0.001 0.001 0.001
- link hip2_1: geometry collision box size=0.1 0.40 0.1; visual mesh filename=package://centauro/centauro_urdf/meshes/simplified/hip-pitc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 scale=0.001 0.001 0.001
- link hip2_2: geometry collision box size=0.1 0.40 0.1; visual mesh filename=package://centauro/centauro_urdf/meshes/simplified/hip-pitc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 scale=0.001 0.001 0.001
- link hip2_3: geometry collision box size=0.1 0.40 0.1; visual mesh filename=package://centauro/centauro_urdf/meshes/simplified/hip-pitc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 scale=0.001 0.001 0.001
- link hip2_4: geometry collision box size=0.1 0.40 0.1; visual mesh filename=package://centauro/centauro_urdf/meshes/simplified/hip-pitc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 scale=0.001 0.001 0.001
- link knee_1: geometry collision box size=0.30 0.1 0.1; visual mesh filename=package://centauro/centauro_urdf/meshes/simplified/knee.stl scale=0.001 0.001 0.001
- link knee_2: geometry collision box size=0.30 0.1 0.1; visual mesh filename=package://centauro/centauro_urdf/meshes/simplified/knee.stl scale=0.001 0.001 0.001
- link knee_3: geometry collision box size=0.30 0.1 0.1; visual mesh filename=package://centauro/centauro_urdf/meshes/simplified/knee.stl scale=0.001 0.001 0.001
- link knee_4: geometry collision box size=0.30 0.1 0.1; visual mesh filename=package://centauro/centauro_urdf/meshes/simplified/knee.stl scale=0.001 0.001 0.001
- link neck_1: geometry visual mesh filename=package://centauro/centauro_urdf/meshes/simplified/neck_yaw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 scale=0.001 0.001 0.001
- link neck_2: geometry visual mesh filename=package://centauro/centauro_urdf/meshes/simplified/neck_pit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 scale=0.001 0.001 0.001
- link neck_3: geometry visual mesh filename=package://centauro/centauro_urdf/meshes/simplified/velodyne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 scale=0.001 0.001 0.001
- link pelvis: geometry collision box size=0.52 0.38 0.25; visual mesh filename=package://centauro/centauro_urdf/meshes/simplified/pelvis.s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 scale=0.001 0.001 0.001
- link torso_2: geometry collision box size=0.1 0.2 0.3; visual mesh filename=package://centauro/centauro_urdf/meshes/simplified/link1.stl scale=0.001 0.001 0.001
- link wheel_1: geometry collision sphere radius=0.078; visual mesh filename=package://centauro/centauro_urdf/meshes/simplified/wheel.stl scale=0.001 0.001 0.001
- link wheel_2: geometry collision sphere radius=0.078; visual mesh filename=package://centauro/centauro_urdf/meshes/simplified/wheel.stl scale=0.001 0.001 0.001
- link wheel_3: geometry collision sphere radius=0.078; visual mesh filename=package://centauro/centauro_urdf/meshes/simplified/wheel.stl scale=0.001 0.001 0.001
- link wheel_4: geometry collision sphere radius=0.078; visual mesh filename=package://centauro/centauro_urdf/meshes/simplified/wheel.stl scale=0.001 0.001 0.001
Joints:
- removed joint j_ft_1
- removed joint j_ft_2
- joint j_arm1_8: origin xyz=0.0 0.0 0.0 rpy=0.0 0.0 0.0 -> xyz=0.0 0.0 -0.0405 rpy=0.0 3.14159265359 -1.5707963268; parent ft_arm1 -> arm1_7
- joint j_arm2_8: origin xyz=0.0 0.0 0.0 rpy=0.0 0.0 -1.5707963268 -> xyz=0.0 0.0 -0.0405 rpy=0.0 3.14159265359 -1.5707963268; parent ft_arm2 -> arm2_7

Commit message: add collision models for fore-arms

File: centauro/urdf/centauro.urdf (robot description, URDF)
Before this commit: robot centauro, 53 links, 52 joints
Links:
- link arm1_7: geometry collision cylinder length=0.15 radius=0.05; visual mesh filename=package://centauro/centauro_urdf/meshes/simplified/link8.stl scale=0.001 -0.001 0.001
- link arm2_7: geometry collision cylinder length=0.15 radius=0.05; visual mesh filename=package://centauro/centauro_urdf/meshes/simplified/link8.stl scale=0.001 0.001 0.001

Commit message: removed the hand mass, to have it compatible with stick EEs

File: centauro/urdf/centauro.urdf (robot description, URDF)
Before this commit: robot centauro, 55 links, 54 joints
Links:
- link arm1_8: mass 1.8366865 -> 0.15; geometry collision mesh filename=package://centauro/centauro_urdf/meshes/convex_hull/link9.s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 scale=0.001 0.001 -0.001; visual mesh filename=package://centauro/centauro_urdf/meshes/simplified/link9.stl scale=0.001 0.001 -0.001

Commit message: Heri Hand successfully integrated, configs to keep!

File: centauro/urdf/centauro.urdf (robot description, URDF)
Before this commit: robot centauro, 53 links, 52 joints
Links:
- added link arm1_9, mass 0.15; collision mesh filename=package://centauro/centauro_urdf/meshes/convex_hull/link9.s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 scale=0.001 -0.001 -0.001; visual mesh filename=package://centauro/centauro_urdf/meshes/simplified/link9.stl scale=0.001 -0.001 -0.001
- added link velodyne, mass 0.0
- added link velodyne_upright, mass 0.0
Joints:
- removed joint j_arm1_8
- added joint 110: type fixed, parent arm1_7, child arm1_8, origin xyz=0.0 0.0 -0.0405 rpy=0.0 3.14159265359 -1.5707963268, axis 1 0 0, limit lower=0.0 upper=0 effort=0 velocity=0
- added joint 111: type fixed, parent arm1_8, child arm1_9, origin xyz=0.0 0.0 -0.0405 rpy=0.0 3.14159265359 -1.5707963268, axis 1 0 0, limit lower=0.0 upper=0 effort=0 velocity=0
- added joint j_velodyne: type fixed, parent neck_3, child velodyne, origin xyz=-0.138 0.0 -0.033 rpy=-1.57079632679 0.0349066 1.57079632679 
- added joint j_velodyne_upright: type fixed, parent velodyne, child velodyne_upright, origin xyz=0.0 0.0 0.0  rpy=1.57079632679 0.0 0.0 

Commit message: larger hip yaw range

File: centauro/urdf/centauro.urdf (robot description, URDF)
Before this commit: robot centauro, 56 links, 55 joints
Joints:
- joint hip_yaw_1: limit lower=-1.13446401 upper=2.70526034 effort=304 velocity=8.8 -> lower=-3.13446401 upper=2.70526034 effort=304 velocity=8.8
- joint hip_yaw_2: limit lower=-2.70526034 upper=1.13446401 effort=304 velocity=8.8 -> lower=-2.70526034 upper=3.13446401 effort=304 velocity=8.8
- joint hip_yaw_3: limit lower=-2.70526034 upper=1.13446401 effort=304 velocity=8.8 -> lower=-2.70526034 upper=3.13446401 effort=304 velocity=8.8
- joint hip_yaw_4: limit lower=-1.13446401 upper=2.70526034 effort=304 velocity=8.8 -> lower=-3.13446401 upper=2.70526034 effort=304 velocity=8.8

Commit message: Latest URDF to check and map on the real robot.

File: centauro/urdf/centauro.urdf (robot description, URDF)
Before this commit: robot centauro, 56 links, 55 joints
Joints:
- joint hip_yaw_1: limit lower=-3.13446401 upper=2.70526034 effort=304 velocity=8.8 -> lower=-2.05 upper=2.48 effort=304 velocity=8.8
- joint hip_yaw_2: limit lower=-2.70526034 upper=3.13446401 effort=304 velocity=8.8 -> lower=-2.48 upper=2.05 effort=304 velocity=8.8
- joint hip_yaw_3: limit lower=-2.70526034 upper=3.13446401 effort=304 velocity=8.8 -> lower=-2.48 upper=2.0 effort=304 velocity=8.8
- joint hip_yaw_4: limit lower=-3.13446401 upper=2.70526034 effort=304 velocity=8.8 -> lower=-2.0 upper=2.48 effort=304 velocity=8.8
