Commit message: updated WALKMAN config files

File: bigman/srdf/bigman.srdf.xacro (robot description, xacro)
@@ -89,6 +89,4 @@
     </group>
     <!-- END F-T sensors -->
-    <!-- TBD IMU -->
-    <!-- TBD END IMU -->
     <!-- Disabled Joint -->
 <!--     <disabled_joint name="LShSag"/> -->

File: bigman/urdf/bigman.urdf (robot description, URDF)
Before this commit: robot bigman, 73 links, 72 joints
Links:
- added link LSoftHandLink, mass 1.2; collision mesh filename=package://bigman_urdf/meshes/simple/SoftHandOpen.STL scale=0.001 -0.001 0.001; visual mesh filename=package://bigman_urdf/meshes/SoftHandOpen.STL scale=0.001 -0.001 0.001
- added link RSoftHandLink, mass 1.2; collision mesh filename=package://bigman_urdf/meshes/simple/SoftHandOpen.STL scale=0.001 0.001 0.001; visual mesh filename=package://bigman_urdf/meshes/SoftHandOpen.STL scale=0.001 0.001 0.001
- added link TCP_L
- added link TCP_R
- added link l_hand_lower_left_link
- added link l_hand_lower_right_link
- added link l_hand_upper_left_link
- added link l_hand_upper_right_link
- added link r_hand_lower_left_link
- added link r_hand_lower_right_link
- added link r_hand_upper_left_link
- added link r_hand_upper_right_link
- link LSoftHand: mass 1.2 -> None; geometry 
- link RSoftHand: mass 1.2 -> None; geometry 
Joints:
- added joint TCP_Ljoint: type fixed, parent LSoftHand, child TCP_L, origin xyz=0.0 0.0 0.0 rpy=1.57079632679 3.14159265359 0
- added joint TCP_Rjoint: type fixed, parent RSoftHand, child TCP_R, origin xyz=0.0 0.0 0.0 rpy=-1.57079632679 0 0
- added joint l_handj2: type fixed, parent LSoftHandLink, child LSoftHand, origin xyz=0 -0.0305 -0.21 rpy=0 0 0
- added joint l_handj3: type fixed, parent LSoftHand, child l_hand_upper_right_link, origin xyz=0.05 0.0 0.0 rpy=0 0 0
- added joint l_handj4: type fixed, parent LSoftHand, child l_hand_lower_right_link, origin xyz=-0.05 0.0 0.0 rpy=0 0 0
- added joint l_handj5: type fixed, parent LSoftHand, child l_hand_upper_left_link, origin xyz=0.05 0.0 0.1 rpy=0 0 0
- added joint l_handj6: type fixed, parent LSoftHand, child l_hand_lower_left_link, origin xyz=-0.05 0.0 0.1 rpy=0 0 0
- added joint r_handj2: type fixed, parent RSoftHandLink, child RSoftHand, origin xyz=0 0.0305 -0.21 rpy=0 0 0
- added joint r_handj3: type fixed, parent RSoftHand, child r_hand_upper_right_link, origin xyz=0.05 0.0 0.0 rpy=0 0 0
- added joint r_handj4: type fixed, parent RSoftHand, child r_hand_lower_right_link, origin xyz=-0.05 0.0 0.0 rpy=0 0 0
- added joint r_handj5: type fixed, parent RSoftHand, child r_hand_upper_left_link, origin xyz=0.05 0.0 0.1 rpy=0 0 0
- added joint r_handj6: type fixed, parent RSoftHand, child r_hand_lower_left_link, origin xyz=-0.05 0.0 0.1 rpy=0 0 0
- joint l_handj: axis -1 0 0 -> (none); child LSoftHand -> LSoftHandLink; limit lower=0 upper=5.0 effort=5 velocity=4.0 -> (none); origin xyz=0 0 -0.04 rpy=0 0 0 -> xyz=0 0 0 rpy=0 0 0; type revolute -> fixed
- joint r_handj: axis 1 0 0 -> (none); child RSoftHand -> RSoftHandLink; limit lower=0.0 upper=5.0 effort=5 velocity=4.0 -> (none); origin xyz=0 0 -0.04 rpy=0 0 0 -> xyz=0 0 0 rpy=0 0 0; type revolute -> fixed
