Commit message: suka

File: kuka/lwr_description/model/kuka_lwr.urdf.xacro (robot description, xacro)
@@ -20,5 +20,5 @@
   <xacro:property name="rate_daming" value="20000"/>
   <!-- URDF model with default base_link (world)-->
-  <xacro:macro name="kuka_lwr" params="name base_link:=world *origin">
+  <xacro:macro name="kuka_lwr" params="name base_link:=world">
     <link name="${base_link}"/>
     <gazebo reference="${base_link}">
@@ -28,5 +28,4 @@
     <!-- First (shoulder) element of the arm. Fixed to its parent. -->
     <joint name="${name}_base_joint" type="fixed">
-      <insert_block name="origin"/>
       <origin xyz="0 0 0" rpy="0 0 0"/>
       <parent link="${base_link}"/>
