Commit message: Updated configs

File: walkman/urdf/walkman.urdf (robot description, URDF)
Before this commit: robot walkman, 33 links, 32 joints
Links:
- added link LElb, mass 1.3157289; collision mesh filename=package://walkman_urdf/meshes/simple/Elbow.STL scale=0.001 -0.001 0.001; visual mesh filename=package://walkman_urdf/meshes/Elbow.STL scale=0.001 -0.001 0.001
- added link LForearm, mass 1.4908547; collision mesh filename=package://walkman_urdf/meshes/simple/Forearm.STL scale=0.001 -0.001 0.001; visual mesh filename=package://walkman_urdf/meshes/Forearm.STL scale=0.001 -0.001 0.001
- added link LShp, mass 1.9628675; collision mesh filename=package://walkman_urdf/meshes/simple/ShoulderPitch.STL scale=0.001 -0.001 0.001; visual mesh filename=package://walkman_urdf/meshes/ShoulderPitch.STL scale=0.001 -0.001 0.001
- added link LShr, mass 1.8595811; collision mesh filename=package://walkman_urdf/meshes/simple/ShoulderRoll.STL scale=0.001 -0.001 0.001; visual mesh filename=package://walkman_urdf/meshes/ShoulderRoll.STL scale=0.001 -0.001 0.001
- added link LShy, mass 1.6678109; collision mesh filename=package://walkman_urdf/meshes/simple/ShoulderYaw.STL scale=0.001 -0.001 0.001; visual mesh filename=package://walkman_urdf/meshes/ShoulderYaw.STL scale=0.001 -0.001 0.001
- added link LWrMot2, mass 1.1263612; collision mesh filename=package://walkman_urdf/meshes/simple/ForearmPitch.STL scale=0.001 -0.001 0.001; visual mesh filename=package://walkman_urdf/meshes/ForearmPitch.STL scale=0.001 -0.001 0.001
- added link LWrMot3, mass 2.7966428e-01; collision mesh filename=package://walkman_urdf/meshes/simple/ForearmYaw.STL scale=0.001 -0.001 0.001; visual mesh filename=package://walkman_urdf/meshes/ForearmYaw.STL scale=0.001 -0.001 0.001
- added link RElb, mass 1.3157289; collision mesh filename=package://walkman_urdf/meshes/simple/Elbow.STL scale=0.001 0.001 0.001; visual mesh filename=package://walkman_urdf/meshes/Elbow.STL scale=0.001 0.001 0.001
- added link RForearm, mass 1.4908547; collision mesh filename=package://walkman_urdf/meshes/simple/Forearm.STL scale=0.001 0.001 0.001; visual mesh filename=package://walkman_urdf/meshes/Forearm.STL scale=0.001 0.001 0.001
- added link RShp, mass 1.9628675; collision mesh filename=package://walkman_urdf/meshes/simple/ShoulderPitch.STL scale=0.001 0.001 0.001; visual mesh filename=package://walkman_urdf/meshes/ShoulderPitch.STL scale=0.001 0.001 0.001
- added link RShr, mass 1.8595811; collision mesh filename=package://walkman_urdf/meshes/simple/ShoulderRoll.STL scale=0.001 0.001 0.001; visual mesh filename=package://walkman_urdf/meshes/ShoulderRoll.STL scale=0.001 0.001 0.001
- added link RShy, mass 1.6678109; collision mesh filename=package://walkman_urdf/meshes/simple/ShoulderYaw.STL scale=0.001 0.001 0.001; visual mesh filename=package://walkman_urdf/meshes/ShoulderYaw.STL scale=0.001 0.001 0.001
- added link RWrMot2, mass 1.1263612; collision mesh filename=package://walkman_urdf/meshes/simple/ForearmPitch.STL scale=0.001 0.001 0.001; visual mesh filename=package://walkman_urdf/meshes/ForearmPitch.STL scale=0.001 0.001 0.001
- added link RWrMot3, mass 2.7966428e-01; collision mesh filename=package://walkman_urdf/meshes/simple/ForearmYaw.STL scale=0.001 0.001 0.001; visual mesh filename=package://walkman_urdf/meshes/ForearmYaw.STL scale=0.001 0.001 0.001
- added link l_wrist
- added link r_wrist
Joints:
- added joint LElbj: type revolute, parent LShy, child LElb, origin xyz=0.045 0.05515 -0.074 rpy=0 0 0, axis 0 1 0, limit lower=-2.96705972838 upper=0.593411945677 effort=120 velocity=6.283
- added joint LForearmPlate: type revolute, parent LElb, child LForearm, origin xyz=-0.015 -0.05515 -0.095 rpy=0 0 0, axis 0 0 1, limit lower=-2.529 upper=2.529 effort=60 velocity=6.283
- added joint LShLat: type revolute, parent LShp, child LShr, origin xyz=-0.09015 0.062 0 rpy=-0.1745327 0 0, axis 1 0 0, limit lower=-3.14159265359 upper=3.14159265359 effort=120 velocity=6.283
- added joint LShSag: type revolute, parent DWYTorso, child LShp, origin xyz=0.0457475 0.169137 0.155126 rpy=0.174533 0 -0.5235988, axis 0 1 0, limit lower=-3.14159265359 upper=3.14159265359 effort=120 velocity=6.283
- added joint LShYaw: type revolute, parent LShr, child LShy, origin xyz=0.09015 0 -0.21815 rpy=0 0 0, axis 0 0 1, limit lower=-3.14159265359 upper=3.14159265359 effort=120 velocity=6.283
- added joint LWrj1: type revolute, parent LForearm, child LWrMot2, origin xyz=0 0.049 -0.156 rpy=0 0 0, axis 0 1 0, limit lower=-1.48 upper=1.48 effort=60 velocity=6.283
- added joint LWrj2: type revolute, parent LWrMot2, child LWrMot3, origin xyz=0 -0.049 -0.174 rpy=0 0 0, axis 0 0 1, limit lower=-1.48 upper=1.48 effort=60 velocity=6.283
- added joint RElbj: type revolute, parent RShy, child RElb, origin xyz=0.045 -0.05515 -0.074 rpy=0 0 0, axis 0 1 0, limit lower=-2.96705972838 upper=0.593411945677 effort=120 velocity=6.283
- added joint RForearmPlate: type revolute, parent RElb, child RForearm, origin xyz=-0.015 0.05515 -0.095 rpy=0 0 0, axis 0 0 1, limit lower=-2.529 upper=2.529 effort=60 velocity=6.283
- added joint RShLat: type revolute, parent RShp, child RShr, origin xyz=-0.09015 -0.062 0 rpy=0.1745327 0 0, axis 1 0 0, limit lower=-3.14159265359 upper=3.14159265359 effort=120 velocity=6.283
- added joint RShSag: type revolute, parent DWYTorso, child RShp, origin xyz=0.0457475 -0.169137 0.155126 rpy=-0.174533 0 0.5235988, axis 0 1 0, limit lower=-3.14159265359 upper=3.14159265359 effort=120 velocity=6.283
- added joint RShYaw: type revolute, parent RShr, child RShy, origin xyz=0.09015 0 -0.21815 rpy=0 0 0, axis 0 0 1, limit lower=-3.14159265359 upper=3.14159265359 effort=120 velocity=6.283
- added joint RWrj1: type revolute, parent RForearm, child RWrMot2, origin xyz=0 -0.049 -0.156 rpy=0 0 0, axis 0 1 0, limit lower=-1.48 upper=1.48 effort=60 velocity=6.283
- added joint RWrj2: type revolute, parent RWrMot2, child RWrMot3, origin xyz=0 0.049 -0.174 rpy=0 0 0, axis 0 0 1, limit lower=-1.48 upper=1.48 effort=60 velocity=6.283
- added joint l_wrist_joint: type fixed, parent LWrMot3, child l_wrist, origin xyz=0 0 0 rpy=0 0 0
- added joint r_wrist_joint: type fixed, parent RWrMot3, child r_wrist, origin xyz=0 0 0 rpy=0 0 0

Commit message: updated urdf

File: walkman/urdf/walkman.urdf (robot description, URDF)
Before this commit: robot walkman, 49 links, 48 joints
Joints:
- joint LAnkLat: limit lower=-0.785 upper=0.785 effort=210 velocity=6.283 -> lower=-0.785398163396 upper=0.785398163396 effort=210 velocity=6.283
- joint LAnkSag: limit lower=-1.39556 upper=0.697778 effort=330 velocity=6.283 -> lower=-1.39626340159 upper=0.698131700796 effort=330 velocity=6.283
- joint LElbj: limit lower=-2.96705972838 upper=0.593411945677 effort=120 velocity=6.283 -> lower=-2.53072741539 upper=0.349065850398 effort=147 velocity=6.283
- joint LForearmPlate: limit lower=-2.529 upper=2.529 effort=60 velocity=6.283 -> lower=-2.61799387799 upper=2.61799387799 effort=55 velocity=6.283
- joint LHipLat: limit lower=-0.697778 upper=0.87222 effort=400 velocity=6.283 -> lower=-0.698131700796 upper=0.872664625995 effort=400 velocity=6.283
- joint LHipSag: limit lower=-2.09333 upper=1.046667 effort=400 velocity=6.283 -> lower=-2.09439510239 upper=1.04719755119 effort=400 velocity=6.283
- joint LHipYaw: limit lower=-0.872222 upper=1.57 effort=140 velocity=6.283 -> lower=-0.872664625995 upper=1.57079632679 effort=140 velocity=6.283
- joint LKneeSag: limit lower=0.0 upper=2.442222 effort=400 velocity=6.283 -> lower=0.0 upper=2.44346095279 effort=400 velocity=6.283
- joint LShLat: limit lower=-3.14159265359 upper=3.14159265359 effort=120 velocity=6.283 -> lower=0 upper=3.49065850398 effort=120 velocity=6.283
- joint LShSag: limit lower=-3.14159265359 upper=3.14159265359 effort=120 velocity=6.283 -> lower=-3.40339204138 upper=1.65806278939 effort=147 velocity=6.283
- joint LShYaw: limit lower=-3.14159265359 upper=3.14159265359 effort=120 velocity=6.283 -> lower=-2.61799387799 upper=2.61799387799 effort=147 velocity=6.283
- joint LWrj1: limit lower=-1.48 upper=1.48 effort=60 velocity=6.283 -> lower=-1.57079632679 upper=1.57079632679 effort=55 velocity=6.283
- joint LWrj2: limit lower=-1.48 upper=1.48 effort=60 velocity=6.283 -> lower=-2.61799387799 upper=2.61799387799 effort=27 velocity=6.283
- joint RAnkLat: limit lower=-0.785 upper=0.785 effort=210 velocity=6.283 -> lower=-0.785398163396 upper=0.785398163396 effort=210 velocity=6.283
- joint RAnkSag: limit lower=-1.39556 upper=0.697778 effort=330 velocity=6.283 -> lower=-1.39626340159 upper=0.698131700796 effort=330 velocity=6.283
- joint RElbj: limit lower=-2.96705972838 upper=0.593411945677 effort=120 velocity=6.283 -> lower=-2.96705972838 upper=0.593411945677 effort=147 velocity=6.283
- joint RForearmPlate: limit lower=-2.529 upper=2.529 effort=60 velocity=6.283 -> lower=-2.61799387799 upper=2.61799387799 effort=55 velocity=6.283
- joint RHipLat: limit lower=-0.87222 upper=0.697778 effort=400 velocity=6.283 -> lower=-0.872664625995 upper=0.698131700796 effort=400 velocity=6.283
- joint RHipSag: limit lower=-2.09333 upper=1.046667 effort=400 velocity=6.283 -> lower=-2.09439510239 upper=1.04719755119 effort=400 velocity=6.283
- joint RHipYaw: limit lower=-1.57 upper=0.872222 effort=140 velocity=6.283 -> lower=-1.57079632679 upper=0.872664625995 effort=140 velocity=6.283
- joint RKneeSag: limit lower=0.0 upper=2.442222 effort=400 velocity=6.283 -> lower=0.0 upper=2.44346095279 effort=400 velocity=6.283
- joint RShLat: limit lower=-3.14159265359 upper=3.14159265359 effort=120 velocity=6.283 -> lower=-3.49065850398 upper=0 effort=120 velocity=6.283
- joint RShSag: limit lower=-3.14159265359 upper=3.14159265359 effort=120 velocity=6.283 -> lower=-3.40339204138 upper=1.65806278939 effort=147 velocity=6.283
- joint RShYaw: limit lower=-3.14159265359 upper=3.14159265359 effort=120 velocity=6.283 -> lower=-2.61799387799 upper=2.61799387799 effort=147 velocity=6.283
- joint RWrj1: limit lower=-1.48 upper=1.48 effort=60 velocity=6.283 -> lower=-1.57079632679 upper=1.57079632679 effort=55 velocity=6.283
- joint RWrj2: limit lower=-1.48 upper=1.48 effort=60 velocity=6.283 -> lower=-2.61799387799 upper=2.61799387799 effort=27 velocity=6.283

Commit message: add imu

File: walkman/urdf/walkman.urdf (robot description, URDF)
Before this commit: robot walkman, 49 links, 48 joints
Links:
- added link imu_link, mass 0.01; visual box size=0.01 0.01 0.01
- added link imu_link2, mass 0.01; visual box size=0.01 0.01 0.01
Joints:
- added joint imu_joint: type fixed, parent Waist, child imu_link, origin xyz=0.0535 0.0 0.0601 rpy=0 0 0
- added joint imu_joint2: type fixed, parent Waist, child imu_link2, origin xyz=0.0135 0.0 0.0601 rpy=0 0 0
- joint LAnkLat: limit lower=-0.785398163396 upper=0.785398163396 effort=210 velocity=6.283 -> lower=-0.785398163398 upper=0.785398163398 effort=210 velocity=6.283
- joint LAnkSag: limit lower=-1.39626340159 upper=0.698131700796 effort=330 velocity=6.283 -> lower=-1.3962634016 upper=0.698131700798 effort=330 velocity=6.283
- joint LElbj: limit lower=-2.53072741539 upper=0.349065850398 effort=147 velocity=6.283 -> lower=-2.53072741539 upper=0.349065850399 effort=147 velocity=6.283
- joint LHipLat: limit lower=-0.698131700796 upper=0.872664625995 effort=400 velocity=6.283 -> lower=-0.698131700798 upper=0.872664625997 effort=400 velocity=6.283
- joint LHipSag: limit lower=-2.09439510239 upper=1.04719755119 effort=400 velocity=6.283 -> lower=-2.09439510239 upper=1.0471975512 effort=400 velocity=6.283
- joint LHipYaw: limit lower=-0.872664625995 upper=1.57079632679 effort=140 velocity=6.283 -> lower=-0.872664625997 upper=1.5707963268 effort=140 velocity=6.283
- joint LShLat: limit lower=0 upper=3.49065850398 effort=120 velocity=6.283 -> lower=0 upper=3.49065850399 effort=120 velocity=6.283
- joint LShSag: limit lower=-3.40339204138 upper=1.65806278939 effort=147 velocity=6.283 -> lower=-3.40339204139 upper=1.65806278939 effort=147 velocity=6.283
- joint LWrj1: limit lower=-1.57079632679 upper=1.57079632679 effort=55 velocity=6.283 -> lower=-1.5707963268 upper=1.5707963268 effort=55 velocity=6.283
- joint NeckPitchj: limit lower=-0.261799387798 upper=1.04719755119 effort=120 velocity=6.283 -> lower=-0.261799387799 upper=1.0471975512 effort=120 velocity=6.283
- joint NeckYawj: limit lower=-0.610865238196 upper=0.610865238196 effort=120 velocity=6.283 -> lower=-0.610865238198 upper=0.610865238198 effort=120 velocity=6.283
- joint RAnkLat: limit lower=-0.785398163396 upper=0.785398163396 effort=210 velocity=6.283 -> lower=-0.785398163398 upper=0.785398163398 effort=210 velocity=6.283
- joint RAnkSag: limit lower=-1.39626340159 upper=0.698131700796 effort=330 velocity=6.283 -> lower=-1.3962634016 upper=0.698131700798 effort=330 velocity=6.283
- joint RElbj: limit lower=-2.96705972838 upper=0.593411945677 effort=147 velocity=6.283 -> lower=-2.96705972839 upper=0.593411945678 effort=147 velocity=6.283
- joint RHipLat: limit lower=-0.872664625995 upper=0.698131700796 effort=400 velocity=6.283 -> lower=-0.872664625997 upper=0.698131700798 effort=400 velocity=6.283
- joint RHipSag: limit lower=-2.09439510239 upper=1.04719755119 effort=400 velocity=6.283 -> lower=-2.09439510239 upper=1.0471975512 effort=400 velocity=6.283
- joint RHipYaw: limit lower=-1.57079632679 upper=0.872664625995 effort=140 velocity=6.283 -> lower=-1.5707963268 upper=0.872664625997 effort=140 velocity=6.283
- joint RShLat: limit lower=-3.49065850398 upper=0 effort=120 velocity=6.283 -> lower=-3.49065850399 upper=0 effort=120 velocity=6.283
- joint RShSag: limit lower=-3.40339204138 upper=1.65806278939 effort=147 velocity=6.283 -> lower=-3.40339204139 upper=1.65806278939 effort=147 velocity=6.283
- joint RWrj1: limit lower=-1.57079632679 upper=1.57079632679 effort=55 velocity=6.283 -> lower=-1.5707963268 upper=1.5707963268 effort=55 velocity=6.283
- joint WaistLat: limit lower=-0.610865238196 upper=0.610865238196 effort=120 velocity=6.283 -> lower=-0.610865238198 upper=0.610865238198 effort=120 velocity=6.283

Commit message: updated urdf and srdf

File: walkman/urdf/walkman.urdf (robot description, URDF)
Before this commit: robot walkman, 49 links, 48 joints
Links:
- added link imu_link, mass 0.01; visual box size=0.01 0.01 0.01
Joints:
- added joint imu_joint: type fixed, parent Waist, child imu_link, origin xyz=0.0 0.0 0.0 rpy=0 0 0

Commit message: Updated urdf

File: walkman/urdf/walkman.urdf (robot description, URDF)
Before this commit: robot walkman, 50 links, 49 joints
Joints:
- joint imu_joint: origin xyz=0.0 0.0 0.0 rpy=0 0 0 -> xyz=0.116998 2.83129e-05 -0.0478857 rpy=0 0 0

Commit message: updated urdf

File: walkman/urdf/walkman.urdf (robot description, URDF)
Before this commit: robot walkman, 50 links, 49 joints
Links:
- added link LSoftHand
- added link LSoftHandLink, mass 1.4; collision mesh filename=package://walkman_urdf/meshes/simple/SoftHandOpen2.STL scale=0.001 -0.001 0.001; visual mesh filename=package://walkman_urdf/meshes/SoftHandOpen2.STL scale=0.001 -0.001 0.001
- added link RSoftHand
- added link RSoftHandLink, mass 1.4; collision mesh filename=package://walkman_urdf/meshes/simple/SoftHandOpen2.STL scale=0.001 0.001 0.001; visual mesh filename=package://walkman_urdf/meshes/SoftHandOpen2.STL scale=0.001 0.001 0.001
- added link TCP_L
- added link TCP_R
- link l_wrist: mass None -> 3.7827821e-01; geometry collision mesh filename=package://walkman_urdf/meshes/simple/Wrist.STL scale=0.001 -0.001 0.001; visual mesh filename=package://walkman_urdf/meshes/Wrist.STL scale=0.001 -0.001 0.001
- link r_wrist: mass None -> 3.7827821e-01; geometry collision mesh filename=package://walkman_urdf/meshes/simple/Wrist.STL scale=0.001 0.001 0.001; visual mesh filename=package://walkman_urdf/meshes/Wrist.STL scale=0.001 0.001 0.001
Joints:
- added joint TCP_Ljoint: type fixed, parent LSoftHand, child TCP_L, origin xyz=0.0 0.0 0.0 rpy=1.57079632679 3.14159265359 0
- added joint TCP_Rjoint: type fixed, parent RSoftHand, child TCP_R, origin xyz=0.0 0.0 0.0 rpy=-1.57079632679 0 0
- added joint l_handj: type fixed, parent l_wrist, child LSoftHandLink, origin xyz=0 0 -0.0395 rpy=0 0 0
- added joint l_handj2: type fixed, parent LSoftHandLink, child LSoftHand, origin xyz=0 -0.041 -0.1005 rpy=0 0 0
- added joint r_handj: type fixed, parent r_wrist, child RSoftHandLink, origin xyz=0 0 -0.0395 rpy=0 0 0
- added joint r_handj2: type fixed, parent RSoftHandLink, child RSoftHand, origin xyz=0 0.041 -0.1005 rpy=0 0 0
- joint LAnkLat: limit lower=-0.785398163396 upper=0.785398163396 effort=210 velocity=6.283 -> lower=-0.785398163398 upper=0.785398163398 effort=210 velocity=6.283
- joint LAnkSag: limit lower=-1.39626340159 upper=0.698131700796 effort=330 velocity=6.283 -> lower=-1.3962634016 upper=0.698131700798 effort=330 velocity=6.283
- joint LElbj: limit lower=-2.53072741539 upper=0.349065850398 effort=147 velocity=6.283 -> lower=-2.492 upper=0.298 effort=147 velocity=6.283
- joint LForearmPlate: limit lower=-2.61799387799 upper=2.61799387799 effort=55 velocity=6.283 -> lower=-2.55 upper=2.55 effort=55 velocity=6.283
- joint LHipLat: limit lower=-0.698131700796 upper=0.872664625995 effort=400 velocity=6.283 -> lower=-0.698131700798 upper=0.872664625997 effort=400 velocity=6.283
- joint LHipSag: limit lower=-2.09439510239 upper=1.04719755119 effort=400 velocity=6.283 -> lower=-2.09439510239 upper=1.0471975512 effort=400 velocity=6.283
- joint LHipYaw: limit lower=-0.872664625995 upper=1.57079632679 effort=140 velocity=6.283 -> lower=-0.872664625997 upper=1.5707963268 effort=140 velocity=6.283
- joint LShLat: limit lower=0 upper=3.49065850398 effort=120 velocity=6.283 -> lower=0.037 upper=3.517 effort=120 velocity=6.283
- joint LShSag: limit lower=-3.40339204138 upper=1.65806278939 effort=147 velocity=6.283 -> lower=-3.352 upper=1.603 effort=147 velocity=6.283
- joint LShYaw: limit lower=-2.61799387799 upper=2.61799387799 effort=147 velocity=6.283 -> lower=-2.55 upper=2.55 effort=147 velocity=6.283
- joint LWrj1: limit lower=-1.57079632679 upper=1.57079632679 effort=55 velocity=6.283 -> lower=-1.562 upper=1.478 effort=55 velocity=6.283
- joint LWrj2: limit lower=-2.61799387799 upper=2.61799387799 effort=27 velocity=6.283 -> lower=-2.55 upper=2.55 effort=27 velocity=6.283
- joint NeckPitchj: limit lower=-0.261799387798 upper=1.04719755119 effort=120 velocity=6.283 -> lower=-0.261799387799 upper=1.0471975512 effort=120 velocity=6.283
- joint NeckYawj: limit lower=-0.610865238196 upper=0.610865238196 effort=120 velocity=6.283 -> lower=-0.610865238198 upper=0.610865238198 effort=120 velocity=6.283
- joint RAnkLat: limit lower=-0.785398163396 upper=0.785398163396 effort=210 velocity=6.283 -> lower=-0.785398163398 upper=0.785398163398 effort=210 velocity=6.283
- joint RAnkSag: limit lower=-1.39626340159 upper=0.698131700796 effort=330 velocity=6.283 -> lower=-1.3962634016 upper=0.698131700798 effort=330 velocity=6.283
- joint RElbj: limit lower=-2.96705972838 upper=0.593411945677 effort=147 velocity=6.283 -> lower=-2.488 upper=0.292 effort=147 velocity=6.283
- joint RForearmPlate: limit lower=-2.61799387799 upper=2.61799387799 effort=55 velocity=6.283 -> lower=-2.55 upper=2.55 effort=55 velocity=6.283
- joint RHipLat: limit lower=-0.872664625995 upper=0.698131700796 effort=400 velocity=6.283 -> lower=-0.872664625997 upper=0.698131700798 effort=400 velocity=6.283
- joint RHipSag: limit lower=-2.09439510239 upper=1.04719755119 effort=400 velocity=6.283 -> lower=-2.09439510239 upper=1.0471975512 effort=400 velocity=6.283
- joint RHipYaw: limit lower=-1.57079632679 upper=0.872664625995 effort=140 velocity=6.283 -> lower=-1.5707963268 upper=0.872664625997 effort=140 velocity=6.283
- joint RShLat: limit lower=-3.49065850398 upper=0 effort=120 velocity=6.283 -> lower=-3.43 upper=-0.004 effort=120 velocity=6.283
- joint RShSag: limit lower=-3.40339204138 upper=1.65806278939 effort=147 velocity=6.283 -> lower=-3.359 upper=1.606 effort=147 velocity=6.283
- joint RShYaw: limit lower=-2.61799387799 upper=2.61799387799 effort=147 velocity=6.283 -> lower=-2.55 upper=2.55 effort=147 velocity=6.283
- joint RWrj1: limit lower=-1.57079632679 upper=1.57079632679 effort=55 velocity=6.283 -> lower=-1.542 upper=1.508 effort=55 velocity=6.283
- joint RWrj2: limit lower=-2.61799387799 upper=2.61799387799 effort=27 velocity=6.283 -> lower=-2.55 upper=2.55 effort=27 velocity=6.283
- joint WaistLat: limit lower=-0.610865238196 upper=0.610865238196 effort=120 velocity=6.283 -> lower=-0.610865238198 upper=0.610865238198 effort=120 velocity=6.283

Commit message: Added FT for the arms

File: walkman/urdf/walkman.urdf (robot description, URDF)
Before this commit: robot walkman, 56 links, 55 joints
Links:
- added link l_arm_ft
- added link r_arm_ft
Joints:
- added joint l_arm_ft_joint: type fixed, parent LWrMot3, child l_arm_ft, origin xyz=0 0 -0.0565 rpy=0 0 0
- added joint r_arm_ft_joint: type fixed, parent RWrMot3, child r_arm_ft, origin xyz=0 0 -0.0565 rpy=0 0 0

Commit message: updated model

File: walkman/urdf/walkman.urdf (robot description, URDF)
Before this commit: robot walkman, 56 links, 55 joints
Links:
- added link l_arm_ft
- added link r_arm_ft
Joints:
- added joint l_arm_ft_joint: type fixed, parent LWrMot3, child l_arm_ft, origin xyz=0 0 -0.0235 rpy=0 0 0
- added joint r_arm_ft_joint: type fixed, parent RWrMot3, child r_arm_ft, origin xyz=0 0 -0.0235 rpy=0 0 0
- joint imu_joint: origin xyz=0.116998 2.83129e-05 -0.0478857 rpy=0 0 0 -> xyz=0.117 0.0 -0.0477493 rpy=0 0 0

Commit message: updated model
Conflicts:
	walkman/urdf/walkman.urdf

File: walkman/urdf/walkman.urdf (robot description, URDF)
Before this commit: robot walkman, 58 links, 57 joints
Joints:
- joint imu_joint: origin xyz=0.116998 2.83129e-05 -0.0478857 rpy=0 0 0 -> xyz=0.117 0.0 -0.0477493 rpy=0 0 0
- joint l_arm_ft_joint: origin xyz=0 0 -0.0565 rpy=0 0 0 -> xyz=0 0 -0.0235 rpy=0 0 0
- joint r_arm_ft_joint: origin xyz=0 0 -0.0565 rpy=0 0 0 -> xyz=0 0 -0.0235 rpy=0 0 0

Commit message: add force torque sensors in hands

File: walkman/urdf/walkman.urdf (robot description, URDF)
Before this commit: robot walkman, 51 links, 50 joints
Links:
- added link l_arm_ft
- added link r_arm_ft
- link LWrMot3: geometry collision box size=0.1 0.1 0.01; visual box size=0.1 0.1 0.01
- link RWrMot3: geometry collision box size=0.1 0.1 0.01; visual box size=0.1 0.1 0.01
Joints:
- added joint l_arm_ft_joint: type fixed, parent LWrMot3, child l_arm_ft, origin xyz=0 0 -0.0565 rpy=0 0 0
- added joint r_arm_ft_joint: type fixed, parent RWrMot3, child r_arm_ft, origin xyz=0 0 -0.0565 rpy=0 0 0

Commit message: updated walkman urdf with gaze frame

File: walkman/urdf/walkman.urdf (robot description, URDF)
Before this commit: robot walkman, 58 links, 57 joints
Links:
- added link gaze
Joints:
- added joint gaze_joint: type fixed, parent NeckPitch, child gaze, origin xyz=0 -0.03425 0 rpy=0 0 0
