Commit message: cogimon simple example working with cogimon whole body (but head)

File: cogimon/urdf/cogimon_lowerbody.urdf (robot description, URDF)
Before this commit: robot cogimon, 51 links, 50 joints
Links:
- removed link DWLExt
- removed link DWYTorso
- removed link LElb
- removed link LForearm
- removed link LShp
- removed link LShr
- removed link LShy
- removed link LWrMot2
- removed link LWrMot3
- removed link RElb
- removed link RForearm
- removed link RShp
- removed link RShr
- removed link RShy
- removed link RWrMot2
- removed link RWrMot3
- removed link imu_link
- added link pennacchio, mass 2.1651618; collision mesh filename=package://cogimon_urdf/meshes/simple/Pennacchio.stl scale=0.001 0.001 0.001; visual mesh filename=package://cogimon_urdf/meshes/Pennacchio.stl scale=0.001 0.001 0.001
- added link weight, mass 30.0; collision cylinder length=0.06 radius=0.055; visual cylinder length=0.06 radius=0.055
Joints:
- removed joint LElbj
- removed joint LForearmPlate
- removed joint LShLat
- removed joint LShSag
- removed joint LShYaw
- removed joint LWrj1
- removed joint LWrj2
- removed joint RElbj
- removed joint RForearmPlate
- removed joint RShLat
- removed joint RShSag
- removed joint RShYaw
- removed joint RWrj1
- removed joint RWrj2
- removed joint WaistFixed
- removed joint WaistYaw
- removed joint imu_joint
- added joint pennacchio_frame: type fixed, parent DWL, child pennacchio, origin xyz=-0.0540957 0.0 0.0665 rpy=0 0 0
- added joint weight_frame: type fixed, parent pennacchio, child weight, origin xyz=0. 0. 0.2 rpy=0 0 0
