Commit message: updated urdf and srdf with ft sensors

File: cogimon/urdf/cogimon.urdf (robot description, URDF)
Before this commit: robot cogimon, 31 links, 30 joints
Links:
- added link l_leg_ft
- added link r_leg_ft
- link LFoot: geometry collision box size=0.21 0.11 0.015; visual mesh filename=model://iit-cogimon/meshes/Foot.stl scale=0.001 0.001 0.001
- link LFootmot: geometry collision mesh filename=model://iit-cogimon/meshes/simple/AnklePitch.stl scale=0.001 0.001 0.001; visual mesh filename=model://iit-cogimon/meshes/AnklePitch.stl scale=0.001 0.001 0.001
- link LHipMot: geometry collision mesh filename=model://iit-cogimon/meshes/simple/HipRoll.stl scale=0.001 0.001 0.001; visual mesh filename=model://iit-cogimon/meshes/HipRoll.stl scale=0.001 0.001 0.001
- link LLowLeg: geometry collision mesh filename=model://iit-cogimon/meshes/simple/KneePitch.stl scale=0.001 0.001 0.001; visual mesh filename=model://iit-cogimon/meshes/KneePitch.stl scale=0.001 0.001 0.001
- link LThighLowLeg: geometry collision mesh filename=model://iit-cogimon/meshes/simple/HipYaw.stl scale=0.001 0.001 0.001; visual mesh filename=model://iit-cogimon/meshes/HipYaw.stl scale=0.001 0.001 0.001
- link LThighUpLeg: geometry collision mesh filename=model://iit-cogimon/meshes/simple/HipPitch.stl scale=0.001 0.001 0.001; visual mesh filename=model://iit-cogimon/meshes/HipPitch.stl scale=0.001 0.001 0.001
- link RFoot: geometry collision box size=0.21 0.11 0.015; visual mesh filename=model://iit-cogimon/meshes/Foot.stl scale=0.001 0.001 0.001
- link RFootmot: geometry collision mesh filename=model://iit-cogimon/meshes/simple/AnklePitch.stl scale=0.001 0.001 0.001; visual mesh filename=model://iit-cogimon/meshes/AnklePitch.stl scale=0.001 0.001 0.001
- link RHipMot: geometry collision mesh filename=model://iit-cogimon/meshes/simple/HipRoll.stl scale=0.001 -0.001 0.001; visual mesh filename=model://iit-cogimon/meshes/HipRoll.stl scale=0.001 -0.001 0.001
- link RLowLeg: geometry collision mesh filename=model://iit-cogimon/meshes/simple/KneePitch.stl scale=0.001 -0.001 0.001; visual mesh filename=model://iit-cogimon/meshes/KneePitch.stl scale=0.001 -0.001 0.001
- link RThighLowLeg: geometry collision mesh filename=model://iit-cogimon/meshes/simple/HipYaw.stl scale=0.001 -0.001 0.001; visual mesh filename=model://iit-cogimon/meshes/HipYaw.stl scale=0.001 -0.001 0.001
- link RThighUpLeg: geometry collision mesh filename=model://iit-cogimon/meshes/simple/HipPitch.stl scale=0.001 -0.001 0.001; visual mesh filename=model://iit-cogimon/meshes/HipPitch.stl scale=0.001 -0.001 0.001
- link Waist: geometry collision mesh filename=model://iit-cogimon/meshes/simple/Waist.stl scale=0.001 0.001 0.001; visual mesh filename=model://iit-cogimon/meshes/Waist.stl scale=0.001 0.001 0.001
Joints:
- added joint l_leg_ft_joint: type fixed, parent LFoot, child l_leg_ft, origin xyz=0 0 -0.035 rpy=0 0 0
- added joint r_leg_ft_joint: type fixed, parent RFoot, child r_leg_ft, origin xyz=0 0 -0.035 rpy=0 0 0

Commit message: Whole legs config working with proper signs

File: cogimon/urdf/cogimon.urdf (robot description, URDF)
Before this commit: robot cogimon, 36 links, 35 joints
Joints:
- joint RAnklePitch: type fixed -> revolute
- joint RAnkleRoll: type fixed -> revolute
- joint RKneePitch: type fixed -> revolute

Commit message: cogimon working at 2ms period with proper current and torque limits.

File: cogimon/urdf/cogimon.urdf (robot description, URDF)
Before this commit: robot cogimon, 51 links, 50 joints
Links:
- added link l_wrist, mass 3.7827821e-01; collision mesh filename=package://walkman_urdf/meshes/simple/Wrist.STL scale=0.001 -0.001 0.001; visual mesh filename=package://walkman_urdf/meshes/Wrist.STL scale=0.001 -0.001 0.001
- added link r_wrist, mass 3.7827821e-01; collision mesh filename=package://walkman_urdf/meshes/simple/Wrist.STL scale=0.001 0.001 0.001; visual mesh filename=package://walkman_urdf/meshes/Wrist.STL scale=0.001 0.001 0.001
Joints:
- added joint l_wrist_joint: type fixed, parent LWrMot3, child l_wrist, origin xyz=0 0 0 rpy=0 0 0
- added joint r_wrist_joint: type fixed, parent RWrMot3, child r_wrist, origin xyz=0 0 0 rpy=0 0 0
- joint LAnklePitch: limit lower=-0.872664625997 upper=0.698131700798 effort=179 velocity=4.9 -> lower=-0.872664625997 upper=0.698131700798 effort=200 velocity=4.9
- joint LAnkleRoll: limit lower=-0.261799387799 upper=0.261799387799 effort=230 velocity=3.2 -> lower=-0.261799387799 upper=0.261799387799 effort=60 velocity=3.2
- joint LElbj: limit lower=-2.492 upper=0.298 effort=147 velocity=6.283 -> lower=-2.492 upper=0.298 effort=120 velocity=6.283
- joint LForearmPlate: limit lower=-2.55 upper=2.55 effort=55 velocity=6.283 -> lower=-2.55 upper=2.55 effort=35 velocity=6.283
- joint LHipLat: limit lower=-0.523598775598 upper=1.65806278939 effort=235 velocity=7.4 -> lower=-0.523598775598 upper=1.65806278939 effort=200 velocity=7.4
- joint LHipSag: limit lower=-1.91986217719 upper=1.55334303428 effort=235 velocity=7.4 -> lower=-1.91986217719 upper=1.55334303428 effort=200 velocity=7.4
- joint LHipYaw: limit lower=-0.558505360638 upper=1.5707963268 effort=153 velocity=4.6 -> lower=-0.558505360638 upper=1.5707963268 effort=120 velocity=4.6
- joint LKneePitch: limit lower=0.0 upper=2.44346095279 effort=313 velocity=5.5 -> lower=0.0 upper=2.44346095279 effort=200 velocity=5.5
- joint LShLat: limit lower=0.037 upper=3.517 effort=120 velocity=6.283 -> lower=0.0 upper=3.517 effort=140 velocity=6.283
- joint LShSag: limit lower=-3.352 upper=1.603 effort=147 velocity=6.283 -> lower=-3.352 upper=1.603 effort=140 velocity=6.283
- joint LShYaw: limit lower=-2.55 upper=2.55 effort=147 velocity=6.283 -> lower=-2.55 upper=2.55 effort=120 velocity=6.283
- joint LWrj1: limit lower=-1.562 upper=1.478 effort=55 velocity=6.283 -> lower=-1.562 upper=1.478 effort=35 velocity=6.283
- joint LWrj2: limit lower=-2.55 upper=2.55 effort=27 velocity=6.283 -> lower=-2.55 upper=2.55 effort=20 velocity=6.283
- joint RAnklePitch: limit lower=-0.872664625997 upper=0.698131700798 effort=179 velocity=4.9 -> lower=-0.872664625997 upper=0.698131700798 effort=200 velocity=4.9
- joint RAnkleRoll: limit lower=-0.261799387799 upper=0.261799387799 effort=230 velocity=3.2 -> lower=-0.261799387799 upper=0.261799387799 effort=60 velocity=3.2
- joint RElbj: limit lower=-2.488 upper=0.292 effort=147 velocity=6.283 -> lower=-2.488 upper=0.292 effort=120 velocity=6.283
- joint RForearmPlate: limit lower=-2.55 upper=2.55 effort=55 velocity=6.283 -> lower=-2.55 upper=2.55 effort=35 velocity=6.283
- joint RHipLat: limit lower=-1.65806278939 upper=0.523598775598 effort=235 velocity=7.4 -> lower=-1.65806278939 upper=0.523598775598 effort=200 velocity=7.4
- joint RHipSag: limit lower=-1.91986217719 upper=1.55334303428 effort=235 velocity=7.4 -> lower=-1.91986217719 upper=1.55334303428 effort=200 velocity=7.4
- joint RHipYaw: limit lower=-1.5707963268 upper=0.558505360638 effort=153 velocity=4.9 -> lower=-1.5707963268 upper=0.558505360638 effort=120 velocity=4.9
- joint RKneePitch: limit lower=0.0 upper=2.44346095279 effort=313 velocity=5.5 -> lower=0.0 upper=2.44346095279 effort=200 velocity=5.5
- joint RShLat: limit lower=-3.43 upper=-0.004 effort=120 velocity=6.283 -> lower=-3.43 upper=0.0 effort=140 velocity=6.283
- joint RShSag: limit lower=-3.359 upper=1.606 effort=147 velocity=6.283 -> lower=-3.359 upper=1.606 effort=140 velocity=6.283
- joint RShYaw: limit lower=-2.55 upper=2.55 effort=147 velocity=6.283 -> lower=-2.55 upper=2.55 effort=120 velocity=6.283
- joint RWrj1: limit lower=-1.542 upper=1.508 effort=55 velocity=6.283 -> lower=-1.542 upper=1.508 effort=35 velocity=6.283
- joint RWrj2: limit lower=-2.55 upper=2.55 effort=27 velocity=6.283 -> lower=-2.55 upper=2.55 effort=20 velocity=6.283
- joint WaistLat: limit lower=-0.523598775598 upper=0.523598775598 effort=150 velocity=7.4 -> lower=-0.523598775598 upper=0.523598775598 effort=140 velocity=7.4

Commit message: imu and head integrated (head to be added back). Tested and working on the real robot

File: cogimon/urdf/cogimon.urdf (robot description, URDF)
Before this commit: robot cogimon, 53 links, 52 joints
Links:
- removed link l_wrist
- removed link r_wrist
- added link HeadHokuyo, mass 5.4611797e-01; collision mesh filename=package://cogimon_urdf/meshes/simple/HeadRoll.stl scale=0.001 0.001 0.001; visual mesh filename=package://cogimon_urdf/meshes/HeadRoll.stl scale=0.001 0.001 0.001
- added link Neck, mass 2.3794941e-01; collision mesh filename=package://cogimon_urdf/meshes/simple/NeckFixed.stl scale=0.001 0.001 0.001; visual mesh filename=package://cogimon_urdf/meshes/NeckFixed.stl scale=0.001 0.001 0.001
Joints:
- removed joint l_wrist_joint
- removed joint r_wrist_joint
- added joint head_roll: type revolute, parent Neck, child HeadHokuyo, origin xyz=0.0496 0.0 0.09 rpy=0 0 0, axis 1 0 0, limit lower=-2.5 upper=2.5 effort=20 velocity=6.283
- added joint neck_frame: type fixed, parent DWYTorso, child Neck, origin xyz=0.016 0.0 0.1965 rpy=0 0 0

Commit message: Full robot working version

File: cogimon/urdf/cogimon.urdf (robot description, URDF)
Before this commit: robot cogimon, 53 links, 52 joints
Links:
- added link LSoftHand
- added link LSoftHandLink, mass 1.4; collision mesh filename=package://cogimon_urdf/meshes/simple/SoftHandOpen2.STL scale=0.001 -0.001 0.001; visual mesh filename=package://cogimon_urdf/meshes/SoftHandOpen2.STL scale=0.001 -0.001 0.001
- added link RSoftHand
- added link RSoftHandLink, mass 1.4; collision mesh filename=package://cogimon_urdf/meshes/simple/SoftHandOpen2.STL scale=0.001 0.001 0.001; visual mesh filename=package://cogimon_urdf/meshes/SoftHandOpen2.STL scale=0.001 0.001 0.001
- added link TCP_L
- added link TCP_R
- added link l_arm_ft
- added link l_wrist, mass 3.7827821e-01; collision mesh filename=package://cogimon_urdf/meshes/simple/Wrist.STL scale=0.001 -0.001 0.001; visual mesh filename=package://cogimon_urdf/meshes/Wrist.STL scale=0.001 -0.001 0.001
- added link r_arm_ft
- added link r_wrist, mass 3.7827821e-01; collision mesh filename=package://cogimon_urdf/meshes/simple/Wrist.STL scale=0.001 0.001 0.001; visual mesh filename=package://cogimon_urdf/meshes/Wrist.STL scale=0.001 0.001 0.001
- link LFoot: mass 1.7819594e+00 -> 2.0663292; geometry collision box size=0.21 0.11 0.015; visual mesh filename=package://cogimon_urdf/meshes/Foot2.stl scale=0.001 0.001 0.001
- link RFoot: mass 1.7819594e+00 -> 2.0663292; geometry collision box size=0.21 0.11 0.015; visual mesh filename=package://cogimon_urdf/meshes/Foot2.stl scale=0.001 0.001 0.001
- link imu_link: mass 0 -> 0.01; geometry visual box size=0.01 0.01 0.01
Joints:
- added joint TCP_Ljoint: type fixed, parent LSoftHand, child TCP_L, origin xyz=0.0 0.0 0.0 rpy=1.57079632679 3.14159265359 0
- added joint TCP_Rjoint: type fixed, parent RSoftHand, child TCP_R, origin xyz=0.0 0.0 0.0 rpy=-1.57079632679 0 0
- added joint l_arm_ft_joint: type fixed, parent LWrMot3, child l_arm_ft, origin xyz=0 0 -0.02 rpy=0 0 0
- added joint l_handj: type fixed, parent l_wrist, child LSoftHandLink, origin xyz=0 0 -0.0395 rpy=0 0 0
- added joint l_handj2: type fixed, parent LSoftHandLink, child LSoftHand, origin xyz=0 -0.041 -0.1005 rpy=0 0 0
- added joint l_wrist_joint: type fixed, parent LWrMot3, child l_wrist, origin xyz=0 0 0 rpy=0 0 0
- added joint r_arm_ft_joint: type fixed, parent RWrMot3, child r_arm_ft, origin xyz=0 0 -0.02 rpy=0 0 0
- added joint r_handj: type fixed, parent r_wrist, child RSoftHandLink, origin xyz=0 0 -0.0395 rpy=0 0 0
- added joint r_handj2: type fixed, parent RSoftHandLink, child RSoftHand, origin xyz=0 0.041 -0.1005 rpy=0 0 0
- added joint r_wrist_joint: type fixed, parent RWrMot3, child r_wrist, origin xyz=0 0 0 rpy=0 0 0
- joint imu_joint: origin xyz=0 0 0 rpy=0 0 0 -> xyz=-0.146332 0 -0.03875 rpy=0 0 0
- joint l_sole_joint: origin xyz=0 0 -0.054 rpy=0 0 0 -> xyz=0 0 -0.069 rpy=0 0 0
- joint r_sole_joint: origin xyz=0 0 -0.054 rpy=0 0 0 -> xyz=0 0 -0.069 rpy=0 0 0
