Commit message: bonn_centauro is the right mesh package

File: bonn_centauro/urdf/bonn_centauro.urdf (robot description, URDF)
Before this commit: robot bonn_centauro, 20 links, 19 joints
Links:
- link DWLExt: geometry collision mesh filename=package://bonn_centauro_urdf/meshes/simple/TorsoRollExt.stl scale=0.001 0.001 0.001; visual mesh filename=package://bonn_centauro_urdf/meshes/TorsoRollExt.stl scale=0.001 0.001 0.001
- link DWYTorso: geometry collision mesh filename=package://bonn_centauro_urdf/meshes/simple/Chest.stl scale=0.001 0.001 0.001; visual mesh filename=package://bonn_centauro_urdf/meshes/Chest.stl scale=0.001 0.001 0.001
- link LElb: geometry collision mesh filename=package://bonn_centauro_urdf/meshes/simple/Elbow.STL scale=0.001 -0.001 0.001; visual mesh filename=package://bonn_centauro_urdf/meshes/Elbow.STL scale=0.001 -0.001 0.001
- link LForearm: geometry collision mesh filename=package://bonn_centauro_urdf/meshes/simple/Forearm.STL scale=0.001 -0.001 0.001; visual mesh filename=package://bonn_centauro_urdf/meshes/Forearm.STL scale=0.001 -0.001 0.001
- link LShp: geometry collision mesh filename=package://bonn_centauro_urdf/meshes/simple/ShoulderPitch.STL scale=0.001 -0.001 0.001; visual mesh filename=package://bonn_centauro_urdf/meshes/ShoulderPitch.STL scale=0.001 -0.001 0.001
- link LShr: geometry collision mesh filename=package://bonn_centauro_urdf/meshes/simple/ShoulderRoll.STL scale=0.001 -0.001 0.001; visual mesh filename=package://bonn_centauro_urdf/meshes/ShoulderRoll.STL scale=0.001 -0.001 0.001
- link LShy: geometry collision mesh filename=package://bonn_centauro_urdf/meshes/simple/ShoulderYaw.STL scale=0.001 -0.001 0.001; visual mesh filename=package://bonn_centauro_urdf/meshes/ShoulderYaw.STL scale=0.001 -0.001 0.001
- link LWrMot2: geometry collision mesh filename=package://bonn_centauro_urdf/meshes/simple/ForearmPitch.STL scale=0.001 -0.001 0.001; visual mesh filename=package://bonn_centauro_urdf/meshes/ForearmPitch.STL scale=0.001 -0.001 0.001
- link LWrMot3: geometry collision mesh filename=package://bonn_centauro_urdf/meshes/simple/ForearmYaw.STL scale=0.001 -0.001 0.001; visual mesh filename=package://bonn_centauro_urdf/meshes/ForearmYaw.STL scale=0.001 -0.001 0.001
- link RElb: geometry collision mesh filename=package://bonn_centauro_urdf/meshes/simple/Elbow.STL scale=0.001 0.001 0.001; visual mesh filename=package://bonn_centauro_urdf/meshes/Elbow.STL scale=0.001 0.001 0.001
- link RForearm: geometry collision mesh filename=package://bonn_centauro_urdf/meshes/simple/Forearm.STL scale=0.001 0.001 0.001; visual mesh filename=package://bonn_centauro_urdf/meshes/Forearm.STL scale=0.001 0.001 0.001
- link RShp: geometry collision mesh filename=package://bonn_centauro_urdf/meshes/simple/ShoulderPitch.STL scale=0.001 0.001 0.001; visual mesh filename=package://bonn_centauro_urdf/meshes/ShoulderPitch.STL scale=0.001 0.001 0.001
- link RShr: geometry collision mesh filename=package://bonn_centauro_urdf/meshes/simple/ShoulderRoll.STL scale=0.001 0.001 0.001; visual mesh filename=package://bonn_centauro_urdf/meshes/ShoulderRoll.STL scale=0.001 0.001 0.001
- link RShy: geometry collision mesh filename=package://bonn_centauro_urdf/meshes/simple/ShoulderYaw.STL scale=0.001 0.001 0.001; visual mesh filename=package://bonn_centauro_urdf/meshes/ShoulderYaw.STL scale=0.001 0.001 0.001
- link RWrMot2: geometry collision mesh filename=package://bonn_centauro_urdf/meshes/simple/ForearmPitch.STL scale=0.001 0.001 0.001; visual mesh filename=package://bonn_centauro_urdf/meshes/ForearmPitch.STL scale=0.001 0.001 0.001
- link RWrMot3: geometry collision mesh filename=package://bonn_centauro_urdf/meshes/simple/ForearmYaw.STL scale=0.001 0.001 0.001; visual mesh filename=package://bonn_centauro_urdf/meshes/ForearmYaw.STL scale=0.001 0.001 0.001
- link Waist: geometry collision mesh filename=package://bonn_centauro_urdf/meshes/simple/Waist.stl scale=0.001 0.001 0.001; visual mesh filename=package://bonn_centauro_urdf/meshes/Waist.stl scale=0.001 0.001 0.001
- link l_wrist: geometry collision mesh filename=package://bonn_centauro_urdf/meshes/simple/Wrist.STL scale=0.001 -0.001 0.001; visual mesh filename=package://bonn_centauro_urdf/meshes/Wrist.STL scale=0.001 -0.001 0.001
- link r_wrist: geometry collision mesh filename=package://bonn_centauro_urdf/meshes/simple/Wrist.STL scale=0.001 0.001 0.001; visual mesh filename=package://bonn_centauro_urdf/meshes/Wrist.STL scale=0.001 0.001 0.001
